File: ProtoBreadboard/ProtoBreadboard.kicad_pcb (KiCad board)
At the start: 2 copper layers, 30.5 x 35.6 mm, 51 parts, among them IC1 BSS138, IC2 BSS138, J1 Conn_01x10_Female, J10 Conn_01x08_Female, J11 Conn_01x06_Female, J12 Conn_01x04_Female, J13 Conn_01x32_Female, J14 Conn_01x32_Female, J15 Conn_01x07_Female, J16 Conn_01x07_Female, J17 AVR-ISP-6, J18 Conn_01x03_Female, J19 Conn_01x02_Female, J2 Conn_01x10_Female, J20 Conn_01x02_Female, J21 Conn_01x15_Female, J22 Conn_01x15_Female, J23 Conn_01x03_Female, J24 Conn_01x02_Female, J25 Conn_01x04_Female, J26 Conn_01x02_Female, J3 Conn_01x30_Female, J4 Conn_01x30_Female, J5 Conn_01x02_Female, J6 Conn_01x02_Female, J7 Conn_01x01_Female, J8 Conn_01x03_Female, J9 Conn_01x08_Female, SW1 RotaryEncoder_Switch, SW2 RotaryEncoder_Switch, U1 60_Pins, U2 PRTR5V0U2X, U3 UG-2864HSWEG01, U4 AP2112K-3.3, Y1 Crystal_GND24_Small

Commit message: Breadboard Mouse Bits
Parts:
- removed AT90USB1286-AU1: 64_Pins, SamacSys_Parts:AT90USB1286-AU
- added G11: Generic_Small, Breadboard:Generic, F.Cu at (47.1, 82.6)
- added G12: Generic_Small, Breadboard:Generic, F.Cu at (47.1, 85.1)
- added G13: Generic_Small, Breadboard:Generic, F.Cu at (47.1, 87.6)
- added G14: Generic_Small, Breadboard:Generic, F.Cu at (47.1, 90.2)
- added G15: Generic_Small, Breadboard:Generic, F.Cu at (47.1, 92.7)
- added G16: Generic_Small, Breadboard:Generic, F.Cu at (47.1, 95.3)
- added G17: Generic_Small, Breadboard:Generic, F.Cu at (47.1, 97.8)
- added G18: Generic_Small, Breadboard:Generic, F.Cu at (47.1, 100.3)
- added G19: Generic_Small, Breadboard:Generic, F.Cu at (47.1, 102.9)
- added G20: Generic_Small, Breadboard:Generic, F.Cu at (47.1, 105.4)
- added G21: Generic_Small, Breadboard:Generic, F.Cu at (65.1, 82.6)
- added G22: Generic_Small, Breadboard:Generic, F.Cu at (65.1, 85.1)
- added G23: Generic_Small, Breadboard:Generic, F.Cu at (65.1, 87.6)
- added G24: Generic_Small, Breadboard:Generic, F.Cu at (65.1, 90.2)
- added G25: Generic_Small, Breadboard:Generic, F.Cu at (65.1, 92.7)
- added G26: Generic_Small, Breadboard:Generic, F.Cu at (65.1, 95.3)
- added G27: Generic_Small, Breadboard:Generic, F.Cu at (65.1, 97.8)
- added G28: Generic_Small, Breadboard:Generic, F.Cu at (65.1, 100.3)
- added G29: Generic_Small, Breadboard:Generic, F.Cu at (65.1, 102.9)
- added G30: Generic_Small, Breadboard:Generic, F.Cu at (65.1, 105.4)
- added G31: Generic_Small, Breadboard:Generic, F.Cu at (83.1, 82.6)
- added G32: Generic_Small, Breadboard:Generic, F.Cu at (83.1, 85.1)
- added G33: Generic_Small, Breadboard:Generic, F.Cu at (83.1, 87.6)
- added G34: Generic_Small, Breadboard:Generic, F.Cu at (83.1, 90.2)
- added G35: Generic_Small, Breadboard:Generic, F.Cu at (83.1, 92.7)
- added G36: Generic_Small, Breadboard:Generic, F.Cu at (83.1, 95.3)
- added G37: Generic_Small, Breadboard:Generic, F.Cu at (83.1, 97.8)
- added G38: Generic_Small, Breadboard:Generic, F.Cu at (83.1, 100.3)
- added G39: Generic_Small, Breadboard:Generic, F.Cu at (83.1, 102.9)
- added G40: Generic_Small, Breadboard:Generic, F.Cu at (83.1, 105.4)
- added G41: Generic_Small, Breadboard:Generic, F.Cu at (101.1, 82.6)
- added G42: Generic_Small, Breadboard:Generic, F.Cu at (101.1, 85.1)
- added G43: Generic_Small, Breadboard:Generic, F.Cu at (101.1, 87.6)
- added G44: Generic_Small, Breadboard:Generic, F.Cu at (101.1, 90.2)
- added G45: Generic_Small, Breadboard:Generic, F.Cu at (101.1, 92.7)
- added G46: Generic_Small, Breadboard:Generic, F.Cu at (101.1, 95.3)
- added G47: Generic_Small, Breadboard:Generic, F.Cu at (101.1, 97.8)
- added G48: Generic_Small, Breadboard:Generic, F.Cu at (101.1, 100.3)
- added G49: Generic_Small, Breadboard:Generic, F.Cu at (101.1, 102.9)
- added G50: Generic_Small, Breadboard:Generic, F.Cu at (101.1, 105.4)
- added G51: Generic_Small, Breadboard:Generic, F.Cu at (119.1, 82.6)
- added G52: Generic_Small, Breadboard:Generic, F.Cu at (119.1, 85.1)
- added G53: Generic_Small, Breadboard:Generic, F.Cu at (119.1, 87.6)
- added G54: Generic_Small, Breadboard:Generic, F.Cu at (119.1, 90.2)
- added G55: Generic_Small, Breadboard:Generic, F.Cu at (119.1, 92.7)
- added G56: Generic_Small, Breadboard:Generic, F.Cu at (119.1, 95.3)
- added G57: Generic_Small, Breadboard:Generic, F.Cu at (119.1, 97.8)
- added G58: Generic_Small, Breadboard:Generic, F.Cu at (119.1, 100.3)
- added G59: Generic_Small, Breadboard:Generic, F.Cu at (119.1, 102.9)
- added G60: Generic_Small, Breadboard:Generic, F.Cu at (119.1, 105.4)
- added IC3: AT90USB1286-AU, SamacSys_Parts:AT90USB1286-AU, F.Cu at (37.2, 166.7)
- added J27: Conn_01x04_Female, Connector_PinHeader_2.54mm:PinHeader_1x04_P2.54mm_Vertical, F.Cu at (123.6, 145.4)
- added J28: Conn_01x10_Female, Connector_PinHeader_2.54mm:PinHeader_1x10_P2.54mm_Vertical, F.Cu at (42.0, 82.6)
- added J29: Conn_01x10_Female, Connector_PinHeader_2.54mm:PinHeader_1x10_P2.54mm_Vertical, F.Cu at (52.2, 82.6)
- added J30: Conn_01x10_Female, Connector_PinHeader_2.54mm:PinHeader_1x10_P2.54mm_Vertical, F.Cu at (60.0, 82.6)
- added J31: Conn_01x10_Female, Connector_PinHeader_2.54mm:PinHeader_1x10_P2.54mm_Vertical, F.Cu at (70.2, 82.6)
- added J32: Conn_01x10_Female, Connector_PinHeader_2.54mm:PinHeader_1x10_P2.54mm_Vertical, F.Cu at (78.0, 82.6)
- added J33: Conn_01x10_Female, Connector_PinHeader_2.54mm:PinHeader_1x10_P2.54mm_Vertical, F.Cu at (88.2, 82.6)
- added J34: Conn_01x10_Female, Connector_PinHeader_2.54mm:PinHeader_1x10_P2.54mm_Vertical, F.Cu at (96.0, 82.6)
- added J35: Conn_01x10_Female, Connector_PinHeader_2.54mm:PinHeader_1x10_P2.54mm_Vertical, F.Cu at (106.2, 82.6)
- added J36: Conn_01x10_Female, Connector_PinHeader_2.54mm:PinHeader_1x10_P2.54mm_Vertical, F.Cu at (114.0, 82.6)
- added J37: Conn_01x10_Female, Connector_PinHeader_2.54mm:PinHeader_1x10_P2.54mm_Vertical, F.Cu at (124.2, 82.6)
- added MX1: MX-NoLED, SamacSys_Parts:MXOnly-1U-NoLED_3Pins, F.Cu at (110.0, 120.8)
- added MX2: MX-NoLED, SamacSys_Parts:MXOnly-1U-NoLED_3Pins, F.Cu at (110.0, 139.9)
- added MX3: MX-NoLED, SamacSys_Parts:MXOnly-1U-NoLED_3Pins, F.Cu at (110.0, 158.9)
- added MX4: MX-NoLED, SamacSys_Parts:MXOnly-1U-NoLED_3Pins, F.Cu at (110.0, 178.0)
- added mouse-bite-2mm-slot: VAL**, Panelization:mouse-bite-2mm-slot, F.Cu at (29.0, 109.0)
- added mouse-bite-2mm-slot: VAL**, Panelization:mouse-bite-2mm-slot, F.Cu at (74.1, 104.0)
- added mouse-bite-2mm-slot: VAL**, Panelization:mouse-bite-2mm-slot, F.Cu at (62.9, 216.0)
- added mouse-bite-2mm-slot: VAL**, Panelization:mouse-bite-2mm-slot, F.Cu at (110.1, 84.0)
- added mouse-bite-2mm-slot: VAL**, Panelization:mouse-bite-2mm-slot, F.Cu at (56.1, 104.0)
- added mouse-bite-2mm-slot: VAL**, Panelization:mouse-bite-2mm-slot, F.Cu at (92.1, 84.0)
- added mouse-bite-2mm-slot: VAL**, Panelization:mouse-bite-2mm-slot, F.Cu at (74.1, 84.0)
- added mouse-bite-2mm-slot: VAL**, Panelization:mouse-bite-2mm-slot, F.Cu at (55.8, 194.2)
- added mouse-bite-2mm-slot: VAL**, Panelization:mouse-bite-2mm-slot, F.Cu at (76.0, 201.0)
- added mouse-bite-2mm-slot: VAL**, Panelization:mouse-bite-2mm-slot, F.Cu at (101.0, 109.0)
- added mouse-bite-2mm-slot: VAL**, Panelization:mouse-bite-2mm-slot, F.Cu at (56.0, 114.0)
- added mouse-bite-2mm-slot: VAL**, Panelization:mouse-bite-2mm-slot, F.Cu at (83.0, 120.0)
- added mouse-bite-2mm-slot: VAL**, Panelization:mouse-bite-2mm-slot, F.Cu at (39.9, 217.0)
- added mouse-bite-2mm-slot: VAL**, Panelization:mouse-bite-2mm-slot, F.Cu at (29.0, 210.0)
- added mouse-bite-2mm-slot: VAL**, Panelization:mouse-bite-2mm-slot, F.Cu at (48.0, 210.0)
- added mouse-bite-2mm-slot: VAL**, Panelization:mouse-bite-2mm-slot, F.Cu at (107.0, 191.0)
- added mouse-bite-2mm-slot: VAL**, Panelization:mouse-bite-2mm-slot, F.Cu at (65.0, 109.0)
- added mouse-bite-2mm-slot: VAL**, Panelization:mouse-bite-2mm-slot, F.Cu at (38.1, 104.0)
- added mouse-bite-2mm-slot: VAL**, Panelization:mouse-bite-2mm-slot, F.Cu at (110.1, 104.0)
- added mouse-bite-2mm-slot: VAL**, Panelization:mouse-bite-2mm-slot, F.Cu at (74.0, 114.0)
- added mouse-bite-2mm-slot: VAL**, Panelization:mouse-bite-2mm-slot, F.Cu at (38.0, 117.0)
- added mouse-bite-2mm-slot: VAL**, Panelization:mouse-bite-2mm-slot, F.Cu at (119.0, 109.0)
- added mouse-bite-2mm-slot: VAL**, Panelization:mouse-bite-2mm-slot, F.Cu at (29.0, 123.0)
- added mouse-bite-2mm-slot: VAL**, Panelization:mouse-bite-2mm-slot, F.Cu at (83.0, 109.0)
- added mouse-bite-2mm-slot: VAL**, Panelization:mouse-bite-2mm-slot, F.Cu at (65.0, 120.0)
- added mouse-bite-2mm-slot: VAL**, Panelization:mouse-bite-2mm-slot, F.Cu at (55.8, 169.0)
- added mouse-bite-2mm-slot: VAL**, Panelization:mouse-bite-2mm-slot, F.Cu at (38.1, 84.0)
- added mouse-bite-2mm-slot: VAL**, Panelization:mouse-bite-2mm-slot, F.Cu at (92.0, 115.0)
- added mouse-bite-2mm-slot: VAL**, Panelization:mouse-bite-2mm-slot, F.Cu at (56.1, 84.0)
- added mouse-bite-2mm-slot: VAL**, Panelization:mouse-bite-2mm-slot, F.Cu at (82.5, 164.0)
- added mouse-bite-2mm-slot: VAL**, Panelization:mouse-bite-2mm-slot, F.Cu at (47.0, 109.0)
- added mouse-bite-2mm-slot: VAL**, Panelization:mouse-bite-2mm-slot, F.Cu at (92.1, 104.0)
- added mouse-bite-2mm-slot: VAL**, Panelization:mouse-bite-2mm-slot, F.Cu at (62.0, 164.0)
- J17: footprint SamacSys_Parts:SWR204NRTND03STGA -> Connector_PinHeader_2.54mm:PinHeader_2x03_P2.54mm_Vertical
- J25: value Conn_01x04_Female -> Conn_01x02_Female; footprint Connector_PinHeader_2.54mm:PinHeader_1x04_P2.54mm_Vertical -> Connector_PinHeader_2.54mm:PinHeader_1x02_P2.54mm_Vertical
- J26: value Conn_01x02_Female -> Conn_01x04_Female; footprint Connector_PinHeader_2.54mm:PinHeader_1x02_P2.54mm_Vertical -> Connector_PinHeader_2.54mm:PinHeader_1x04_P2.54mm_Vertical
- J7: value Conn_01x01_Female -> Conn_01x04_Female; footprint Connector_PinHeader_2.54mm:PinHeader_1x01_P2.54mm_Vertical -> Connector_PinHeader_2.54mm:PinHeader_1x04_P2.54mm_Vertical
- U1: value 60_Pins -> IS31FL3741-QFLS4-TR; footprint SamacSys_Parts:QFN40P700X700X80-61N-D -> Breadboard:IS31FL3741-QFLS4-TR
- moved RGB1 201.9 mm to (76.9, 207.0)
- moved J11 200.2 mm to (59.5, 176.3)
- moved J12 200.2 mm to (84.9, 178.8)
- moved SW1 200.2 mm to (64.9, 171.2)
- moved SW2 200.2 mm to (64.9, 187.7)
- moved RGB2 200.1 mm to (76.9, 212.6)
- moved J10 200.0 mm to (84.7, 206.2)
- moved J9 200.0 mm to (66.9, 206.2)
- moved RGB3 198.1 mm to (76.9, 218.0)
- moved RGB4 196.7 mm to (76.9, 224.0)
- moved J15 181.1 mm to (21.1, 229.3)
- moved J16 181.1 mm to (36.4, 214.0)
- moved USB1 181.1 mm to (28.8, 233.3)
- moved J18 176.4 mm to (59.0, 214.1)
- moved J8 176.4 mm to (43.8, 214.1)
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Connections:
- net Net-(J17-Pad6) renamed GND_6
- net Net-(J23-Pad2) renamed GND_4
- net Net-(U2-Pad1) renamed GND_5
- J13 pad 22: Net-(AT90USB1286-AU1-Pad22) -> GND_1
- J14 pad 21: Net-(AT90USB1286-AU1-Pad53) -> GND_1
- J14 pad 31: Net-(AT90USB1286-AU1-Pad63) -> GND_1
- J15 pad 1: Net-(J15-Pad1) -> GND_2
- J16 pad 5: Net-(J16-Pad5) -> GND_2
- J21 pad 15: Net-(J21-Pad15) -> GND_7
- J22 pad 1: Net-(J22-Pad1) -> GND_7
- J25 pad 1: Net-(IC1-Pad1) -> Net-(IC1-Pad3)
- J25 pad 2: Net-(IC1-Pad2) -> Net-(IC2-Pad3)
- J26 pad 1: Net-(IC1-Pad3) -> Net-(IC1-Pad1)
- J26 pad 2: Net-(IC2-Pad3) -> Net-(IC1-Pad2)
- J3 pad 12: Net-(J3-Pad12) -> GND_3
- J4 pad 25: Net-(J4-Pad25) -> GND_3
- J4 pad 6: Net-(J4-Pad6) -> GND_3
- U1 pad 12: Net-(J3-Pad12) -> GND_3
- U1 pad 36: Net-(J4-Pad6) -> GND_3
- U1 pad 55: Net-(J4-Pad25) -> GND_3
- U1 pad 61: Net-(J7-Pad1) -> GND_3
- U3 pad 1: Net-(J22-Pad1) -> GND_7
- U3 pad 30: Net-(J21-Pad15) -> GND_7
- USB1 pad 1: Net-(J15-Pad1) -> GND_2
- USB1 pad 12: Net-(J16-Pad5) -> GND_2
Routing:
- net GND_3: track 0.00 -> 72.4 mm
- net GND_1: track 0.00 -> 65.5 mm
- net Net-(J13-Pad1): track 0.00 -> 41.7 mm
- net GND_7: track 0.00 -> 41.2 mm
- net Net-(J14-Pad32): track 0.00 -> 41.0 mm
- net Net-(J3-Pad1): track 0.00 -> 39.6 mm
- net Net-(J4-Pad30): track 0.00 -> 39.5 mm
- net Net-(J13-Pad2): track 0.00 -> 39.0 mm
- net Net-(J27-Pad1): track 0.00 -> 38.9 mm
- net Net-(J4-Pad1): track 0.00 -> 37.7 mm
- net Net-(J3-Pad30): track 0.00 -> 37.7 mm
- net Net-(J3-Pad2): track 0.00 -> 37.2 mm
- net Net-(J4-Pad29): track 0.00 -> 37.0 mm
- net Net-(J13-Pad3): track 0.00 -> 36.1 mm
- net Net-(J13-Pad32): track 0.00 -> 35.6 mm
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- added copper zone on B.Cu, net GND_1
- added copper zone on F.Cu, net GND_1
- added copper zone on B.Cu, net GND_2
- added copper zone on F.Cu, net GND_2
- added copper zone on B.Cu, net GND_3
- added copper zone on F.Cu, net GND_3
- added copper zone on B.Cu, net GND_4
- added copper zone on F.Cu, net GND_4
- added copper zone on B.Cu, net GND_5
- added copper zone on F.Cu, net GND_5
- added copper zone on B.Cu, net GND_6
- added copper zone on F.Cu, net GND_6
- added copper zone on B.Cu, net GND_7
- added copper zone on F.Cu, net GND_7
Other:
- board size 30.5 x 35.6 mm -> 108.3 x 194 mm

Commit message: Almost Finished Panelizing
Parts:
- added G1: Generic_Small, Breadboard:Generic, F.Cu at (44.9, 255.6)
- added G1: Generic_Small, Breadboard:Generic, F.Cu at (26.8, 255.6)
- added G1: Generic_Small, Breadboard:Generic, F.Cu at (81.2, 255.6)
- added G1: Generic_Small, Breadboard:Generic, F.Cu at (63.1, 255.6)
- added G10: Generic_Small, Breadboard:Generic, F.Cu at (81.2, 278.4)
- added G10: Generic_Small, Breadboard:Generic, F.Cu at (44.9, 278.4)
- added G10: Generic_Small, Breadboard:Generic, F.Cu at (63.1, 278.4)
- added G10: Generic_Small, Breadboard:Generic, F.Cu at (26.8, 278.4)
- added G2: Generic_Small, Breadboard:Generic, F.Cu at (63.1, 258.1)
- added G2: Generic_Small, Breadboard:Generic, F.Cu at (81.2, 258.1)
- added G2: Generic_Small, Breadboard:Generic, F.Cu at (26.8, 258.1)
- added G2: Generic_Small, Breadboard:Generic, F.Cu at (44.9, 258.1)
- added G3: Generic_Small, Breadboard:Generic, F.Cu at (81.2, 260.6)
- added G3: Generic_Small, Breadboard:Generic, F.Cu at (44.9, 260.6)
- added G3: Generic_Small, Breadboard:Generic, F.Cu at (63.1, 260.6)
- added G3: Generic_Small, Breadboard:Generic, F.Cu at (26.8, 260.6)
- added G4: Generic_Small, Breadboard:Generic, F.Cu at (44.9, 263.2)
- added G4: Generic_Small, Breadboard:Generic, F.Cu at (63.1, 263.2)
- added G4: Generic_Small, Breadboard:Generic, F.Cu at (81.2, 263.2)
- added G4: Generic_Small, Breadboard:Generic, F.Cu at (26.8, 263.2)
- added G5: Generic_Small, Breadboard:Generic, F.Cu at (63.1, 265.7)
- added G5: Generic_Small, Breadboard:Generic, F.Cu at (44.9, 265.7)
- added G5: Generic_Small, Breadboard:Generic, F.Cu at (81.2, 265.7)
- added G5: Generic_Small, Breadboard:Generic, F.Cu at (26.8, 265.7)
- added G6: Generic_Small, Breadboard:Generic, F.Cu at (63.1, 268.3)
- added G6: Generic_Small, Breadboard:Generic, F.Cu at (44.9, 268.3)
- added G6: Generic_Small, Breadboard:Generic, F.Cu at (26.8, 268.3)
- added G6: Generic_Small, Breadboard:Generic, F.Cu at (81.2, 268.3)
- added G7: Generic_Small, Breadboard:Generic, F.Cu at (44.9, 270.8)
- added G7: Generic_Small, Breadboard:Generic, F.Cu at (81.2, 270.8)
- added G7: Generic_Small, Breadboard:Generic, F.Cu at (63.1, 270.8)
- added G7: Generic_Small, Breadboard:Generic, F.Cu at (26.8, 270.8)
- added G8: Generic_Small, Breadboard:Generic, F.Cu at (63.1, 273.3)
- added G8: Generic_Small, Breadboard:Generic, F.Cu at (44.9, 273.3)
- added G8: Generic_Small, Breadboard:Generic, F.Cu at (81.2, 273.3)
- added G8: Generic_Small, Breadboard:Generic, F.Cu at (26.8, 273.3)
- added G9: Generic_Small, Breadboard:Generic, F.Cu at (26.8, 275.9)
- added G9: Generic_Small, Breadboard:Generic, F.Cu at (44.9, 275.9)
- added G9: Generic_Small, Breadboard:Generic, F.Cu at (81.2, 275.9)
- added G9: Generic_Small, Breadboard:Generic, F.Cu at (63.1, 275.9)
- added IC1: BSS138, SamacSys_Parts:SOT95P240X120-3N, F.Cu at (44.7, 241.9)
- added IC2: BSS138, SamacSys_Parts:SOT95P240X120-3N, F.Cu at (44.7, 247.0)
- added J1: Conn_01x10_Female, Connector_PinHeader_2.54mm:PinHeader_1x10_P2.54mm_Vertical, F.Cu at (39.9, 255.6)
- added J1: Conn_01x10_Female, Connector_PinHeader_2.54mm:PinHeader_1x10_P2.54mm_Vertical, F.Cu at (21.7, 255.6)
- added J1: Conn_01x10_Female, Connector_PinHeader_2.54mm:PinHeader_1x10_P2.54mm_Vertical, F.Cu at (58.0, 255.6)
- added J1: Conn_01x10_Female, Connector_PinHeader_2.54mm:PinHeader_1x10_P2.54mm_Vertical, F.Cu at (76.1, 255.6)
- added J17: AVR-ISP-6, Connector_PinHeader_2.54mm:PinHeader_2x03_P2.54mm_Vertical, F.Cu at (50.2, 227.1)
- added J18: Conn_01x03_Female, Connector_PinHeader_2.54mm:PinHeader_1x03_P2.54mm_Vertical, F.Cu at (59.0, 227.1)
- added J19: Conn_01x02_Female, Connector_PinHeader_2.54mm:PinHeader_1x02_P2.54mm_Vertical, F.Cu at (57.6, 240.2)
- added J2: Conn_01x10_Female, Connector_PinHeader_2.54mm:PinHeader_1x10_P2.54mm_Vertical, F.Cu at (31.9, 255.6)
- added J2: Conn_01x10_Female, Connector_PinHeader_2.54mm:PinHeader_1x10_P2.54mm_Vertical, F.Cu at (86.3, 255.6)
- added J2: Conn_01x10_Female, Connector_PinHeader_2.54mm:PinHeader_1x10_P2.54mm_Vertical, F.Cu at (68.2, 255.6)
- added J2: Conn_01x10_Female, Connector_PinHeader_2.54mm:PinHeader_1x10_P2.54mm_Vertical, F.Cu at (50.0, 255.6)
- added J20: Conn_01x02_Female, Connector_PinHeader_2.54mm:PinHeader_1x02_P2.54mm_Vertical, F.Cu at (67.8, 242.8)
- added J23: Conn_01x03_Female, Connector_PinHeader_2.54mm:PinHeader_1x03_P2.54mm_Vertical, F.Cu at (21.7, 238.6)
- added J24: Conn_01x02_Female, Connector_PinHeader_2.54mm:PinHeader_1x02_P2.54mm_Vertical, F.Cu at (31.8, 241.2)
- added J25: Conn_01x02_Female, Connector_PinHeader_2.54mm:PinHeader_1x02_P2.54mm_Vertical, F.Cu at (49.8, 241.5)
- added J26: Conn_01x04_Female, Connector_PinHeader_2.54mm:PinHeader_1x04_P2.54mm_Vertical, F.Cu at (39.7, 240.3)
- added J5: Conn_01x02_Female, Connector_PinHeader_2.54mm:PinHeader_1x02_P2.54mm_Vertical, F.Cu at (75.7, 240.0)
- added J6: Conn_01x02_Female, Connector_PinHeader_2.54mm:PinHeader_1x02_P2.54mm_Vertical, F.Cu at (85.8, 242.6)
- added J8: Conn_01x03_Female, Connector_PinHeader_2.54mm:PinHeader_1x03_P2.54mm_Vertical, F.Cu at (43.8, 227.1)
- added U2: PRTR5V0U2X, random-keyboard-parts:SOT143B, F.Cu at (62.7, 242.0)
- added U4: AP2112K-3.3, SamacSys_Parts:SOT95P282X130-5N, F.Cu at (26.7, 241.2)
- added Y1: Crystal_GND24_Small, Crystal:Crystal_SMD_3225-4Pin_3.2x2.5mm, F.Cu at (80.7, 241.1)
- added mouse-bite-2mm-slot: VAL**, Panelization:mouse-bite-2mm-slot-1-side, F.Cu at (100.2, 215.0)
- added mouse-bite-2mm-slot: VAL**, Panelization:mouse-bite-2mm-slot, F.Cu at (122.0, 191.0)
- added mouse-bite-2mm-slot: VAL**, Panelization:mouse-bite-2mm-slot-1-side, F.Cu at (27.0, 248.0)
- added mouse-bite-2mm-slot: VAL**, Panelization:mouse-bite-2mm-slot-1-side, F.Cu at (81.0, 235.9)
- added mouse-bite-2mm-slot: VAL**, Panelization:mouse-bite-2mm-slot, F.Cu at (39.9, 228.0)
- added mouse-bite-2mm-slot: VAL**, Panelization:mouse-bite-2mm-slot, F.Cu at (72.3, 257.0)
- added mouse-bite-2mm-slot: VAL**, Panelization:mouse-bite-2mm-slot-1-side, F.Cu at (89.8, 241.3)
- added mouse-bite-2mm-slot: VAL**, Panelization:mouse-bite-2mm-slot-1-side, F.Cu at (100.2, 262.3)
- added mouse-bite-2mm-slot: VAL**, Panelization:mouse-bite-2mm-slot, F.Cu at (46.1, 236.0)
- added mouse-bite-2mm-slot: VAL**, Panelization:mouse-bite-2mm-slot-1-side, F.Cu at (92.0, 179.0)
- added mouse-bite-2mm-slot: VAL**, Panelization:mouse-bite-2mm-slot, F.Cu at (35.8, 242.0)
- added mouse-bite-2mm-slot: VAL**, Panelization:mouse-bite-2mm-slot, F.Cu at (26.8, 234.0)
- added mouse-bite-2mm-slot: VAL**, Panelization:mouse-bite-2mm-slot, F.Cu at (54.1, 276.4)
- added mouse-bite-2mm-slot: VAL**, Panelization:mouse-bite-2mm-slot, F.Cu at (44.9, 251.0)
- added mouse-bite-2mm-slot: VAL**, Panelization:mouse-bite-2mm-slot, F.Cu at (58.3, 236.0)
- added mouse-bite-2mm-slot: VAL**, Panelization:mouse-bite-2mm-slot-1-side, F.Cu at (90.4, 262.3)
- added mouse-bite-2mm-slot: VAL**, Panelization:mouse-bite-2mm-slot-1-side, F.Cu at (26.9, 251.1)
- added mouse-bite-2mm-slot: VAL**, Panelization:mouse-bite-2mm-slot, F.Cu at (51.4, 223.0)
- added mouse-bite-2mm-slot: VAL**, Panelization:mouse-bite-2mm-slot-1-side, F.Cu at (62.5, 247.0)
- added mouse-bite-2mm-slot: VAL**, Panelization:mouse-bite-2mm-slot-1-side, F.Cu at (81.0, 229.0)
- added mouse-bite-2mm-slot: VAL**, Panelization:mouse-bite-2mm-slot, F.Cu at (53.8, 241.3)
- added mouse-bite-2mm-slot: VAL**, Panelization:mouse-bite-2mm-slot-1-side, F.Cu at (81.3, 246.9)
- added mouse-bite-2mm-slot: VAL**, Panelization:mouse-bite-2mm-slot, F.Cu at (36.0, 257.0)
- added mouse-bite-2mm-slot: VAL**, Panelization:mouse-bite-2mm-slot-1-side, F.Cu at (88.9, 215.0)
- added mouse-bite-2mm-slot: VAL**, Panelization:mouse-bite-2mm-slot, F.Cu at (72.3, 276.4)
- added mouse-bite-2mm-slot: VAL**, Panelization:mouse-bite-2mm-slot-1-side, F.Cu at (81.0, 251.1)
- added mouse-bite-2mm-slot: VAL**, Panelization:mouse-bite-2mm-slot, F.Cu at (54.1, 257.0)
- added mouse-bite-2mm-slot: VAL**, Panelization:mouse-bite-2mm-slot-1-side, F.Cu at (62.3, 251.1)
- added mouse-bite-2mm-slot: VAL**, Panelization:mouse-bite-2mm-slot, F.Cu at (36.0, 276.4)
- added mouse-bite-2mm-slot: VAL**, Panelization:mouse-bite-2mm-slot, F.Cu at (71.8, 240.9)
- added mouse-bite-2mm-slot: VAL**, Panelization:mouse-bite-2mm-slot-1-side, F.Cu at (100.2, 241.2)
- added mouse-bite-2mm-slot: VAL**, Panelization:mouse-bite-2mm-slot-1-side, F.Cu at (88.8, 179.0)
- moved J3 8.00 mm to (104.0, 195.9)
- moved J4 8.00 mm to (124.3, 269.6)
- moved U1 8.00 mm to (114.2, 231.5)
Routing:
- net Net-(J17-Pad5): track 18.1 -> 36.2 mm
- net Net-(G9-Pad1): track 22.2 -> 36.9 mm
- net Net-(G8-Pad1): track 22.2 -> 36.9 mm
- net Net-(G7-Pad1): track 22.2 -> 36.9 mm
- net Net-(G6-Pad1): track 22.2 -> 36.9 mm
- net Net-(G5-Pad1): track 22.2 -> 36.9 mm
- net Net-(G4-Pad1): track 22.2 -> 36.9 mm
- net Net-(G3-Pad1): track 22.2 -> 36.9 mm
- net Net-(G2-Pad1): track 22.2 -> 36.9 mm
- net Net-(G10-Pad1): track 22.2 -> 36.9 mm
- net Net-(G1-Pad1): track 22.2 -> 36.9 mm
- net Net-(G9-Pad2): track 21.9 -> 36.4 mm
- net Net-(G7-Pad2): track 21.9 -> 36.4 mm
- net Net-(G6-Pad2): track 21.9 -> 36.4 mm
- net Net-(G5-Pad2): track 21.9 -> 36.4 mm
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Other:
- board size 108.3 x 194 mm -> 108.4 x 202 mm

Commit message: Mouse Bits Finished
Parts:
- U4: renamed from U1; value IS31FL3741-QFLS4-TR -> QFN40P700X700X80-61N-D; footprint Breadboard:IS31FL3741-QFLS4-TR -> SamacSys_Parts:QFN40P700X700X80-61N-D
- moved mouse-bite-57 0.27 mm to (81.3, 251.0)
- moved mouse-bite-56 0.21 mm to (62.5, 251.0)
- moved mouse-bite-54 0.15 mm to (27.0, 251.0)
- moved mouse-bite-49 0.10 mm to (100.2, 241.3)
- renumbered G32 to G10, G10 to G100, G42 to G11, G52 to G12, G3 to G13, G13 to G14, G23 to G15, G33 to G16, G43 to G17, G53 to G18, G4 to G19, G11 to G2, G14 to G20, G24 to G21, G34 to G22, G44 to G23, G54 to G24, G5 to G25, G15 to G26, G25 to G27, G35 to G28, G45 to G29, G21 to G3, G55 to G30, G6 to G31, G16 to G32, G26 to G33, G36 to G34, G46 to G35, G56 to G36, G7 to G37, G17 to G38, G27 to G39, G31 to G4, G37 to G40, G47 to G41, G57 to G42, G8 to G43, G18 to G44, G28 to G45, G38 to G46, G48 to G47, G58 to G48, G9 to G49, G41 to G5, G19 to G50, G29 to G51, G39 to G52, G49 to G53, G59 to G54, G10 to G55, G20 to G56, G30 to G57, G40 to G58, G50 to G59, G51 to G6, G1 to G61, G1 to G62, G1 to G63, G1 to G64, G2 to G65, G2 to G66, G2 to G67, G2 to G68, G3 to G69, G2 to G7, G3 to G70, G3 to G71, G3 to G72, G4 to G73, G4 to G74, G4 to G75, G4 to G76, G5 to G77, G5 to G78, G5 to G79, G12 to G8, G5 to G80, G6 to G81, G6 to G82, G6 to G83, G6 to G84, G7 to G85, G7 to G86, G7 to G87, G7 to G88, G8 to G89, G22 to G9, G8 to G90, G8 to G91, G8 to G92, G9 to G93, G9 to G94, G9 to G95, G9 to G96, G10 to G97, G10 to G98, G10 to G99, IC1 to IC4, IC2 to IC5, J35 to J10, J36 to J11, J37 to J12, J5 to J13, J19 to J14, J26 to J15, J23 to J16, J25 to J17, J6 to J18, J20 to J19, J24 to J20, J13 to J23, J7 to J24, J27 to J25, J11 to J26, J12 to J27, J3 to J28, J14 to J29, J28 to J3, J9 to J30, J10 to J31, J16 to J32, J8 to J33, J17 to J34, J18 to J35, J8 to J36, J17 to J37, J18 to J38, J15 to J39, J29 to J4, J23 to J40, J5 to J41, J19 to J42, J26 to J43, J24 to J44, J25 to J45, J6 to J46, J20 to J47, J1 to J48, J2 to J49, J30 to J5, J1 to J50, J2 to J51, J1 to J52, J2 to J53, J1 to J54, J2 to J55, J4 to J56, J31 to J6, J32 to J7, J33 to J8, J34 to J9, U2 to U1, U4 to U2, U4 to U5, U2 to U6, Y1 to Y2, mouse-bite-2mm-slot to mouse-bite-1, mouse-bite-2mm-slot to mouse-bite-10, mouse-bite-2mm-slot to mouse-bite-11, mouse-bite-2mm-slot to mouse-bite-12, mouse-bite-2mm-slot to mouse-bite-13, mouse-bite-2mm-slot to mouse-bite-14, mouse-bite-2mm-slot to mouse-bite-15, mouse-bite-2mm-slot to mouse-bite-16, mouse-bite-2mm-slot to mouse-bite-17, mouse-bite-2mm-slot to mouse-bite-18, mouse-bite-2mm-slot to mouse-bite-19, mouse-bite-2mm-slot to mouse-bite-2, mouse-bite-2mm-slot to mouse-bite-20, mouse-bite-2mm-slot to mouse-bite-21, mouse-bite-2mm-slot to mouse-bite-22, mouse-bite-2mm-slot to mouse-bite-23, mouse-bite-2mm-slot to mouse-bite-24, mouse-bite-2mm-slot to mouse-bite-25, mouse-bite-2mm-slot to mouse-bite-26, mouse-bite-2mm-slot to mouse-bite-27, mouse-bite-2mm-slot to mouse-bite-28, mouse-bite-2mm-slot to mouse-bite-29, mouse-bite-2mm-slot to mouse-bite-3, mouse-bite-2mm-slot to mouse-bite-30, mouse-bite-2mm-slot to mouse-bite-31, mouse-bite-2mm-slot to mouse-bite-32, mouse-bite-2mm-slot to mouse-bite-33, mouse-bite-2mm-slot to mouse-bite-34, mouse-bite-2mm-slot to mouse-bite-35, mouse-bite-2mm-slot to mouse-bite-36, mouse-bite-2mm-slot to mouse-bite-37, mouse-bite-2mm-slot to mouse-bite-38, mouse-bite-2mm-slot to mouse-bite-39, mouse-bite-2mm-slot to mouse-bite-4, mouse-bite-2mm-slot to mouse-bite-40, mouse-bite-2mm-slot to mouse-bite-41, mouse-bite-2mm-slot to mouse-bite-42, mouse-bite-2mm-slot to mouse-bite-43, mouse-bite-2mm-slot to mouse-bite-44, mouse-bite-2mm-slot to mouse-bite-45, mouse-bite-2mm-slot to mouse-bite-46, mouse-bite-2mm-slot to mouse-bite-47, mouse-bite-2mm-slot to mouse-bite-48, mouse-bite-2mm-slot to mouse-bite-49, mouse-bite-2mm-slot to mouse-bite-5, mouse-bite-2mm-slot to mouse-bite-50, mouse-bite-2mm-slot to mouse-bite-51, mouse-bite-2mm-slot to mouse-bite-52, mouse-bite-2mm-slot to mouse-bite-53, mouse-bite-2mm-slot to mouse-bite-54, mouse-bite-2mm-slot to mouse-bite-55, mouse-bite-2mm-slot to mouse-bite-56, mouse-bite-2mm-slot to mouse-bite-57, mouse-bite-2mm-slot to mouse-bite-58, mouse-bite-2mm-slot to mouse-bite-59, mouse-bite-2mm-slot to mouse-bite-6, mouse-bite-2mm-slot to mouse-bite-60, mouse-bite-2mm-slot to mouse-bite-61, mouse-bite-2mm-slot to mouse-bite-62, mouse-bite-2mm-slot to mouse-bite-63, mouse-bite-2mm-slot to mouse-bite-64, mouse-bite-2mm-slot to mouse-bite-65, mouse-bite-2mm-slot to mouse-bite-7, mouse-bite-2mm-slot to mouse-bite-8, mouse-bite-2mm-slot to mouse-bite-9
Routing:
- net GND_4: track 0.00 -> 7.66 mm
- net Net-(J17-Pad5): track 36.2 -> 29.9 mm
Other:
- outline, holes or cut-outs redrawn
- board text added: "1"
- board text added: "10"
- board text added: "11"
- board text added: "12"
- board text added: "13"
- board text added: "14"
- board text added: "15"
- board text added: "16"
- board text added: "17"
- board text added: "18"
- board text added: "19"
- board text added: "2"
- board text added: "20"
- board text added: "3"
- board text added: "4"
- board text added: "5"
- board text added: "6"
- board text added: "7"
- board text added: "8"
- board text added: "9"

Commit message: Updated but something wrong
Parts:
- Y1, Y2: value Crystal_GND24_Small -> Crystal
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- renumbered J21 to JOLED1, J22 to JOLED2, U3 to UOLED1
Connections:
- G10 pad 1: Net-(G2-Pad1) -> Net-(G10-Pad1)
- G10 pad 2: Net-(G2-Pad2) -> Net-(G10-Pad2)
- G2 pad 1: Net-(G1-Pad1) -> Net-(G2-Pad1)
- G2 pad 2: Net-(G1-Pad2) -> Net-(G2-Pad2)
- G3 pad 1: Net-(G1-Pad1) -> Net-(G3-Pad1)
- G3 pad 2: Net-(G1-Pad2) -> Net-(G3-Pad2)
- G4 pad 1: Net-(G1-Pad1) -> Net-(G4-Pad1)
- G4 pad 2: Net-(G1-Pad2) -> Net-(G4-Pad2)
- G5 pad 1: Net-(G1-Pad1) -> Net-(G5-Pad1)
- G5 pad 2: Net-(G1-Pad2) -> Net-(G5-Pad2)
- G6 pad 1: Net-(G1-Pad1) -> Net-(G6-Pad1)
- G6 pad 2: Net-(G1-Pad2) -> Net-(G6-Pad2)
- G7 pad 1: Net-(G2-Pad1) -> Net-(G7-Pad1)
- G7 pad 2: Net-(G2-Pad2) -> Net-(G7-Pad2)
- G8 pad 1: Net-(G2-Pad1) -> Net-(G8-Pad1)
- G8 pad 2: Net-(G2-Pad2) -> Net-(G8-Pad2)
- G9 pad 1: Net-(G2-Pad1) -> Net-(G9-Pad1)
- G9 pad 2: Net-(G2-Pad2) -> Net-(G9-Pad2)
- IC3 pad 1: Net-(J13-Pad1) -> Net-(IC3-Pad1)
- IC3 pad 10: Net-(J13-Pad10) -> Net-(IC3-Pad10)
- IC3 pad 11: Net-(J13-Pad11) -> Net-(IC3-Pad11)
- IC3 pad 12: Net-(J13-Pad12) -> Net-(IC3-Pad12)
- IC3 pad 13: Net-(J13-Pad13) -> Net-(IC3-Pad13)
- IC3 pad 14: Net-(J13-Pad14) -> Net-(IC3-Pad14)
- IC3 pad 15: Net-(J13-Pad15) -> Net-(IC3-Pad15)
- IC3 pad 16: Net-(J13-Pad16) -> Net-(IC3-Pad16)
- IC3 pad 17: Net-(J13-Pad17) -> Net-(IC3-Pad17)
- IC3 pad 18: Net-(J13-Pad18) -> Net-(IC3-Pad18)
- IC3 pad 19: Net-(J13-Pad19) -> Net-(IC3-Pad19)
- IC3 pad 2: Net-(J13-Pad2) -> Net-(IC3-Pad2)
- IC3 pad 20: Net-(J13-Pad20) -> Net-(IC3-Pad20)
- IC3 pad 23: Net-(J13-Pad23) -> Net-(IC3-Pad23)
- IC3 pad 24: Net-(J13-Pad24) -> Net-(IC3-Pad24)
- IC3 pad 25: Net-(J13-Pad25) -> Net-(IC3-Pad25)
- IC3 pad 26: Net-(J13-Pad26) -> Net-(IC3-Pad26)
- IC3 pad 27: Net-(J13-Pad27) -> Net-(IC3-Pad27)
- IC3 pad 28: Net-(J13-Pad28) -> Net-(IC3-Pad28)
- IC3 pad 29: Net-(J13-Pad29) -> Net-(IC3-Pad29)
- IC3 pad 3: Net-(J13-Pad3) -> Net-(IC3-Pad3)
- IC3 pad 30: Net-(J13-Pad30) -> Net-(IC3-Pad30)
- IC3 pad 31: Net-(J13-Pad31) -> Net-(IC3-Pad31)
- IC3 pad 32: Net-(J13-Pad32) -> Net-(IC3-Pad32)
- IC3 pad 33: Net-(J14-Pad1) -> Net-(IC3-Pad33)
- IC3 pad 34: Net-(J14-Pad2) -> Net-(IC3-Pad34)
- IC3 pad 35: Net-(J14-Pad3) -> Net-(IC3-Pad35)
- IC3 pad 36: Net-(J14-Pad4) -> Net-(IC3-Pad36)
- IC3 pad 37: Net-(J14-Pad5) -> Net-(IC3-Pad37)
- IC3 pad 38: Net-(J14-Pad6) -> Net-(IC3-Pad38)
- IC3 pad 39: Net-(J14-Pad7) -> Net-(IC3-Pad39)
- IC3 pad 4: Net-(J13-Pad4) -> Net-(IC3-Pad4)
- IC3 pad 40: Net-(J14-Pad8) -> Net-(IC3-Pad40)
- IC3 pad 41: Net-(J14-Pad9) -> Net-(IC3-Pad41)
- IC3 pad 42: Net-(J14-Pad10) -> Net-(IC3-Pad42)
- IC3 pad 43: Net-(J14-Pad11) -> Net-(IC3-Pad43)
- IC3 pad 44: Net-(J14-Pad12) -> Net-(IC3-Pad44)
- IC3 pad 45: Net-(J14-Pad13) -> Net-(IC3-Pad45)
- IC3 pad 46: Net-(J14-Pad14) -> Net-(IC3-Pad46)
- IC3 pad 47: Net-(J14-Pad15) -> Net-(IC3-Pad47)
- IC3 pad 48: Net-(J14-Pad16) -> Net-(IC3-Pad48)
- IC3 pad 49: Net-(J14-Pad17) -> Net-(IC3-Pad49)
- IC3 pad 5: Net-(J13-Pad5) -> Net-(IC3-Pad5)
- IC3 pad 50: Net-(J14-Pad18) -> Net-(IC3-Pad50)
- IC3 pad 51: Net-(J14-Pad19) -> Net-(IC3-Pad51)
- IC3 pad 52: Net-(J14-Pad20) -> Net-(IC3-Pad52)
- IC3 pad 54: Net-(J14-Pad22) -> Net-(IC3-Pad54)
- IC3 pad 55: Net-(J14-Pad23) -> Net-(IC3-Pad55)
- IC3 pad 56: Net-(J14-Pad24) -> Net-(IC3-Pad56)
- IC3 pad 57: Net-(J14-Pad25) -> Net-(IC3-Pad57)
- IC3 pad 58: Net-(J14-Pad26) -> Net-(IC3-Pad58)
- IC3 pad 59: Net-(J14-Pad27) -> Net-(IC3-Pad59)
- IC3 pad 6: Net-(J13-Pad6) -> Net-(IC3-Pad6)
- IC3 pad 60: Net-(J14-Pad28) -> Net-(IC3-Pad60)
- IC3 pad 61: Net-(J14-Pad29) -> Net-(IC3-Pad61)
- IC3 pad 62: Net-(J14-Pad30) -> Net-(IC3-Pad62)
- IC3 pad 64: Net-(J14-Pad32) -> Net-(IC3-Pad64)
- IC3 pad 7: Net-(J13-Pad7) -> Net-(IC3-Pad7)
- IC3 pad 8: Net-(J13-Pad8) -> Net-(IC3-Pad8)
- IC3 pad 9: Net-(J13-Pad9) -> Net-(IC3-Pad9)
- J10 pad 1: Net-(G1-Pad2) -> Net-(J10-Pad1)
- J10 pad 10: Net-(G10-Pad2) -> (no net)
- J10 pad 2: Net-(G2-Pad2) -> Net-(J10-Pad2)
- J10 pad 3: Net-(G3-Pad2) -> Net-(J10-Pad3)
- J10 pad 4: Net-(G4-Pad2) -> Net-(J10-Pad4)
- J10 pad 5: Net-(G5-Pad2) -> Net-(J10-Pad5)
- J10 pad 6: Net-(G6-Pad2) -> Net-(J10-Pad6)
- J10 pad 7: Net-(G7-Pad2) -> Net-(J10-Pad7)
- J10 pad 8: Net-(G8-Pad2) -> Net-(J10-Pad8)
- J10 pad 9: Net-(G9-Pad2) -> (no net)
- J11 pad 1: Net-(G1-Pad1) -> Net-(J11-Pad1)
- J11 pad 10: Net-(G10-Pad1) -> (no net)
- J11 pad 2: Net-(G2-Pad1) -> Net-(J11-Pad2)
- J11 pad 3: Net-(G3-Pad1) -> Net-(J11-Pad3)
- J11 pad 4: Net-(G4-Pad1) -> Net-(J11-Pad4)
- J11 pad 5: Net-(G5-Pad1) -> Net-(J11-Pad5)
- J11 pad 6: Net-(G6-Pad1) -> Net-(J11-Pad6)
- J11 pad 7: Net-(G7-Pad1) -> (no net)
- J11 pad 8: Net-(G8-Pad1) -> (no net)
- J11 pad 9: Net-(G9-Pad1) -> (no net)
- J12 pad 1: Net-(G1-Pad2) -> Net-(J12-Pad1)
- J12 pad 10: Net-(G10-Pad2) -> (no net)
- J12 pad 2: Net-(G2-Pad2) -> Net-(J12-Pad2)
- J12 pad 3: Net-(G3-Pad2) -> Net-(J12-Pad3)
- J12 pad 4: Net-(G4-Pad2) -> Net-(J12-Pad4)
- J12 pad 5: Net-(G5-Pad2) -> (no net)
- J12 pad 6: Net-(G6-Pad2) -> (no net)
- J12 pad 7: Net-(G7-Pad2) -> (no net)
- J12 pad 8: Net-(G8-Pad2) -> (no net)
- J12 pad 9: Net-(G9-Pad2) -> (no net)
- J13 pad 1: Net-(J5-Pad1) -> Net-(IC3-Pad1)
- J13 pad 2: Net-(J5-Pad2) -> Net-(IC3-Pad2)
- J14 pad 1: GND_5 -> Net-(IC3-Pad33)
- J14 pad 2: Net-(J19-Pad2) -> Net-(IC3-Pad34)
- J15 pad 1: Net-(IC1-Pad1) -> GND_2
- J15 pad 2: Net-(IC1-Pad2) -> Net-(J15-Pad2)
- J15 pad 3: Net-(IC2-Pad1) -> Net-(J15-Pad3)
- J15 pad 4: Net-(IC2-Pad2) -> Net-(J15-Pad4)
- J16 pad 1: Net-(J23-Pad1) -> Net-(J16-Pad1)
- J16 pad 2: GND_4 -> Net-(J16-Pad2)
- J16 pad 3: Net-(J23-Pad3) -> Net-(J16-Pad3)
- J18 pad 1: Net-(J6-Pad1) -> Net-(J17-Pad4)
- J18 pad 2: Net-(J6-Pad2) -> Net-(J17-Pad5)
- J19 pad 1: Net-(J20-Pad1) -> GND_5
- J19 pad 2: Net-(J20-Pad2) -> Net-(J19-Pad2)
- J20 pad 1: Net-(J24-Pad1) -> Net-(J20-Pad1)
- J20 pad 2: Net-(J24-Pad2) -> Net-(J20-Pad2)
- J23 pad 1: Net-(J13-Pad1) -> Net-(J23-Pad1)
- J23 pad 10: Net-(J13-Pad10) -> (no net)
- J23 pad 11: Net-(J13-Pad11) -> (no net)
- J23 pad 12: Net-(J13-Pad12) -> (no net)
- J23 pad 13: Net-(J13-Pad13) -> (no net)
- J23 pad 14: Net-(J13-Pad14) -> (no net)
- J23 pad 15: Net-(J13-Pad15) -> (no net)
- J23 pad 16: Net-(J13-Pad16) -> (no net)
- J23 pad 17: Net-(J13-Pad17) -> (no net)
- J23 pad 18: Net-(J13-Pad18) -> (no net)
- J23 pad 19: Net-(J13-Pad19) -> (no net)
- J23 pad 2: Net-(J13-Pad2) -> GND_4
- J23 pad 20: Net-(J13-Pad20) -> (no net)
- J23 pad 21: Net-(IC3-Pad21) -> (no net)
- J23 pad 22: GND_1 -> (no net)
- J23 pad 23: Net-(J13-Pad23) -> (no net)
- J23 pad 24: Net-(J13-Pad24) -> (no net)
- J23 pad 25: Net-(J13-Pad25) -> (no net)
- J23 pad 26: Net-(J13-Pad26) -> (no net)
- J23 pad 27: Net-(J13-Pad27) -> (no net)
- J23 pad 28: Net-(J13-Pad28) -> (no net)
- J23 pad 29: Net-(J13-Pad29) -> (no net)
- J23 pad 3: Net-(J13-Pad3) -> Net-(J23-Pad3)
- J23 pad 30: Net-(J13-Pad30) -> (no net)
- J23 pad 31: Net-(J13-Pad31) -> (no net)
- J23 pad 32: Net-(J13-Pad32) -> (no net)
- J23 pad 4: Net-(J13-Pad4) -> (no net)
- J23 pad 5: Net-(J13-Pad5) -> (no net)
- J23 pad 6: Net-(J13-Pad6) -> (no net)
- J23 pad 7: Net-(J13-Pad7) -> (no net)
- J23 pad 8: Net-(J13-Pad8) -> (no net)
- J23 pad 9: Net-(J13-Pad9) -> (no net)
- J24 pad 1: Net-(J7-Pad1) -> Net-(J24-Pad1)
- J24 pad 2: Net-(J7-Pad2) -> Net-(J24-Pad2)
- J24 pad 3: Net-(J7-Pad3) -> (no net)
- J24 pad 4: Net-(J7-Pad4) -> (no net)
- J25 pad 1: Net-(J27-Pad1) -> Net-(IC1-Pad3)
- J25 pad 2: Net-(J27-Pad2) -> Net-(IC2-Pad3)
- J25 pad 3: Net-(J27-Pad3) -> (no net)
- J25 pad 4: Net-(J27-Pad4) -> (no net)
- J26 pad 1: Net-(J11-Pad1) -> Net-(IC1-Pad1)
- J26 pad 2: Net-(J11-Pad2) -> Net-(IC1-Pad2)
- J26 pad 3: Net-(J11-Pad3) -> Net-(IC2-Pad1)
- J26 pad 4: Net-(J11-Pad4) -> Net-(IC2-Pad2)
- J26 pad 5: Net-(J11-Pad5) -> (no net)
- J26 pad 6: Net-(J11-Pad6) -> (no net)
- J27 pad 1: Net-(J12-Pad1) -> Net-(J27-Pad1)
- J27 pad 2: Net-(J12-Pad2) -> Net-(J27-Pad2)
- J27 pad 3: Net-(J12-Pad3) -> Net-(J27-Pad3)
- J27 pad 4: Net-(J12-Pad4) -> Net-(J27-Pad4)
- J3 pad 1: Net-(G1-Pad1) -> Net-(J3-Pad1)
- J3 pad 10: Net-(G10-Pad1) -> Net-(J3-Pad10)
- J3 pad 2: Net-(G2-Pad1) -> Net-(J3-Pad2)
- J3 pad 3: Net-(G3-Pad1) -> Net-(J3-Pad3)
- J3 pad 4: Net-(G4-Pad1) -> Net-(J3-Pad4)
- J3 pad 5: Net-(G5-Pad1) -> Net-(J3-Pad5)
- J3 pad 6: Net-(G6-Pad1) -> Net-(J3-Pad6)
- J3 pad 7: Net-(G7-Pad1) -> Net-(J3-Pad7)
- J3 pad 8: Net-(G8-Pad1) -> Net-(J3-Pad8)
- J3 pad 9: Net-(G9-Pad1) -> Net-(J3-Pad9)
- J4 pad 1: Net-(G1-Pad2) -> Net-(J4-Pad1)
- J4 pad 10: Net-(G10-Pad2) -> Net-(J4-Pad10)
- J4 pad 2: Net-(G2-Pad2) -> Net-(J4-Pad2)
- J4 pad 3: Net-(G3-Pad2) -> Net-(J4-Pad3)
- J4 pad 4: Net-(G4-Pad2) -> Net-(J4-Pad4)
- J4 pad 5: Net-(G5-Pad2) -> Net-(J4-Pad5)
- J4 pad 6: Net-(G6-Pad2) -> GND_3
- J4 pad 7: Net-(G7-Pad2) -> Net-(J4-Pad7)
- J4 pad 8: Net-(G8-Pad2) -> Net-(J4-Pad8)
- J4 pad 9: Net-(G9-Pad2) -> Net-(J4-Pad9)
- J5 pad 1: Net-(G1-Pad1) -> Net-(J5-Pad1)
- J5 pad 10: Net-(G10-Pad1) -> (no net)
- J5 pad 2: Net-(G2-Pad1) -> Net-(J5-Pad2)
- J5 pad 3: Net-(G3-Pad1) -> (no net)
- J5 pad 4: Net-(G4-Pad1) -> (no net)
- J5 pad 5: Net-(G5-Pad1) -> (no net)
- J5 pad 6: Net-(G6-Pad1) -> (no net)
- J5 pad 7: Net-(G7-Pad1) -> (no net)
- J5 pad 8: Net-(G8-Pad1) -> (no net)
- J5 pad 9: Net-(G9-Pad1) -> (no net)
- J6 pad 1: Net-(G1-Pad2) -> Net-(J6-Pad1)
- J6 pad 10: Net-(G10-Pad2) -> (no net)
- J6 pad 2: Net-(G2-Pad2) -> Net-(J6-Pad2)
- J6 pad 3: Net-(G3-Pad2) -> (no net)
- J6 pad 4: Net-(G4-Pad2) -> (no net)
- J6 pad 5: Net-(G5-Pad2) -> (no net)
- J6 pad 6: Net-(G6-Pad2) -> (no net)
- J6 pad 7: Net-(G7-Pad2) -> (no net)
- J6 pad 8: Net-(G8-Pad2) -> (no net)
- J6 pad 9: Net-(G9-Pad2) -> (no net)
- J7 pad 1: Net-(G1-Pad1) -> Net-(J7-Pad1)
- J7 pad 10: Net-(G10-Pad1) -> (no net)
- J7 pad 2: Net-(G2-Pad1) -> Net-(J7-Pad2)
- J7 pad 3: Net-(G3-Pad1) -> Net-(J7-Pad3)
- J7 pad 4: Net-(G4-Pad1) -> Net-(J7-Pad4)
- J7 pad 5: Net-(G5-Pad1) -> (no net)
- J7 pad 6: Net-(G6-Pad1) -> (no net)
- J7 pad 7: Net-(G7-Pad1) -> (no net)
- J7 pad 8: Net-(G8-Pad1) -> (no net)
- J7 pad 9: Net-(G9-Pad1) -> (no net)
- J8 pad 1: Net-(G1-Pad2) -> Net-(J17-Pad1)
- J8 pad 10: Net-(G10-Pad2) -> (no net)
- J8 pad 2: Net-(G2-Pad2) -> Net-(J17-Pad2)
- J8 pad 3: Net-(G3-Pad2) -> Net-(J17-Pad3)
- J8 pad 4: Net-(G4-Pad2) -> (no net)
- J8 pad 5: Net-(G5-Pad2) -> (no net)
- J8 pad 6: Net-(G6-Pad2) -> (no net)
- J8 pad 7: Net-(G7-Pad2) -> (no net)
- J8 pad 8: Net-(G8-Pad2) -> (no net)
- J8 pad 9: Net-(G9-Pad2) -> (no net)
- J9 pad 1: Net-(G1-Pad1) -> Net-(J9-Pad1)
- J9 pad 10: Net-(G10-Pad1) -> (no net)
- J9 pad 2: Net-(G2-Pad1) -> Net-(J9-Pad2)
- J9 pad 3: Net-(G3-Pad1) -> Net-(J9-Pad3)
- J9 pad 4: Net-(G4-Pad1) -> Net-(J9-Pad4)
- J9 pad 5: Net-(G5-Pad1) -> Net-(J9-Pad5)
- J9 pad 6: Net-(G6-Pad1) -> Net-(J9-Pad6)
- J9 pad 7: Net-(G7-Pad1) -> Net-(J9-Pad7)
- J9 pad 8: Net-(G8-Pad1) -> Net-(J9-Pad8)
- J9 pad 9: Net-(G9-Pad1) -> (no net)
- U1 pad 1: GND_5 -> Net-(J3-Pad1)
- U1 pad 2: Net-(J19-Pad2) -> Net-(J3-Pad2)
- U1 pad 3: Net-(J20-Pad1) -> Net-(J3-Pad3)
- U1 pad 4: Net-(J20-Pad2) -> Net-(J3-Pad4)
- U2 pad 1: Net-(J23-Pad1) -> GND_5
- U2 pad 2: GND_4 -> Net-(J19-Pad2)
- U2 pad 3: Net-(J23-Pad3) -> Net-(J20-Pad1)
- U2 pad 4: Net-(J24-Pad1) -> Net-(J20-Pad2)
- U2 pad 5: Net-(J24-Pad2) -> (no net)
- U4 pad 1: Net-(J3-Pad1) -> Net-(J23-Pad1)
- U4 pad 10: Net-(J3-Pad10) -> (no net)
- U4 pad 11: Net-(J3-Pad11) -> (no net)
- U4 pad 12: GND_3 -> (no net)
- U4 pad 13: Net-(J3-Pad13) -> (no net)
- U4 pad 14: Net-(J3-Pad14) -> (no net)
- U4 pad 15: Net-(J3-Pad15) -> (no net)
- U4 pad 16: Net-(J3-Pad16) -> (no net)
- U4 pad 17: Net-(J3-Pad17) -> (no net)
- U4 pad 18: Net-(J3-Pad18) -> (no net)
- U4 pad 19: Net-(J3-Pad19) -> (no net)
- U4 pad 2: Net-(J3-Pad2) -> GND_4
- U4 pad 20: Net-(J3-Pad20) -> (no net)
- U4 pad 21: Net-(J3-Pad21) -> (no net)
- U4 pad 22: Net-(J3-Pad22) -> (no net)
- U4 pad 23: Net-(J3-Pad23) -> (no net)
- U4 pad 24: Net-(J3-Pad24) -> (no net)
- U4 pad 25: Net-(J3-Pad25) -> (no net)
- U4 pad 26: Net-(J3-Pad26) -> (no net)
- U4 pad 27: Net-(J3-Pad27) -> (no net)
- U4 pad 28: Net-(J3-Pad28) -> (no net)
- U4 pad 29: Net-(J3-Pad29) -> (no net)
- U4 pad 3: Net-(J3-Pad3) -> Net-(J23-Pad3)
- U4 pad 30: Net-(J3-Pad30) -> (no net)
- U4 pad 31: Net-(J4-Pad1) -> (no net)
- U4 pad 32: Net-(J4-Pad2) -> (no net)
- U4 pad 33: Net-(J4-Pad3) -> (no net)
- U4 pad 34: Net-(J4-Pad4) -> (no net)
- U4 pad 35: Net-(J4-Pad5) -> (no net)
- U4 pad 36: GND_3 -> (no net)
- U4 pad 37: Net-(J4-Pad7) -> (no net)
- U4 pad 38: Net-(J4-Pad8) -> (no net)
- U4 pad 39: Net-(J4-Pad9) -> (no net)
- U4 pad 4: Net-(J3-Pad4) -> Net-(J24-Pad1)
- U4 pad 40: Net-(J4-Pad10) -> (no net)
- U4 pad 41: Net-(J4-Pad11) -> (no net)
- U4 pad 42: Net-(J4-Pad12) -> (no net)
- U4 pad 43: Net-(J4-Pad13) -> (no net)
- U4 pad 44: Net-(J4-Pad14) -> (no net)
- U4 pad 45: Net-(J4-Pad15) -> (no net)
- U4 pad 46: Net-(J4-Pad16) -> (no net)
- U4 pad 47: Net-(J4-Pad17) -> (no net)
- U4 pad 48: Net-(J4-Pad18) -> (no net)
- U4 pad 49: Net-(J4-Pad19) -> (no net)
- U4 pad 5: Net-(J3-Pad5) -> Net-(J24-Pad2)
- U4 pad 50: Net-(J4-Pad20) -> (no net)
- U4 pad 51: Net-(J4-Pad21) -> (no net)
- U4 pad 52: Net-(J4-Pad22) -> (no net)
- U4 pad 53: Net-(J4-Pad23) -> (no net)
- U4 pad 54: Net-(J4-Pad24) -> (no net)
- U4 pad 55: GND_3 -> (no net)
- U4 pad 56: Net-(J4-Pad26) -> (no net)
- U4 pad 57: Net-(J4-Pad27) -> (no net)
- U4 pad 58: Net-(J4-Pad28) -> (no net)
- U4 pad 59: Net-(J4-Pad29) -> (no net)
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Routing:
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Other:
- board text added: "21"
- board text added: "22"
- board text added: "23"
- board text added: "24"
- board text added: "25"
- board text added: "26"
- board text added: "27"
- board text added: "28"
- board text added: "29"
- board text added: "30"
- board text added: "A"
- board text added: "B"
- board text added: "C"
- board text added: "NC"
