File: ProtoBreadboard/ProtoBreadboard.kicad_sch (KiCad schematic)
At the start: 51 parts, among them IC1 BSS138, IC2 BSS138, J1 Conn_01x10_Female, J10 Conn_01x08_Female, J11 Conn_01x06_Female, J12 Conn_01x04_Female, J13 Conn_01x32_Female, J14 Conn_01x32_Female, J15 Conn_01x07_Female, J16 Conn_01x07_Female, J17 AVR-ISP-6, J18 Conn_01x03_Female, J19 Conn_01x02_Female, J2 Conn_01x10_Female, J20 Conn_01x02_Female, J21 Conn_01x15_Female, J22 Conn_01x15_Female, J23 Conn_01x03_Female, J24 Conn_01x02_Female, J25 Conn_01x02_Female, J26 Conn_01x04_Female, J3 Conn_01x30_Female, J4 Conn_01x30_Female, J5 Conn_01x02_Female, J6 Conn_01x02_Female, J7 Conn_01x01_Female, J8 Conn_01x03_Female, J9 Conn_01x08_Female, SW1 RotaryEncoder_Switch, SW2 RotaryEncoder_Switch, U1 60_Pins, U2 PRTR5V0U2X, U3 UG-2864HSWEG01, U4 AP2112K-3.3, Y1 Crystal_GND24_Small

Commit message: Breadboard Mouse Bits
Parts:
- removed AT90USB1286-AU1: 64_Pins, SamacSys_Parts:AT90USB1286-AU, symbol Breadbord:64_Pins
- removed J7: Conn_01x01_Female, Connector_PinHeader_2.54mm:PinHeader_1x01_P2.54mm_Vertical, symbol Connector:Conn_01x01_Female
- removed U1: 60_Pins, SamacSys_Parts:QFN40P700X700X80-61N-D, symbol Breadbord:60_Pins
- added IC3: AT90USB1286-AU, SamacSys_Parts:AT90USB1286-AU, symbol SamacSys_Parts:AT90USB1286-AU
- added J27, J7: Conn_01x04_Female, Connector_PinHeader_2.54mm:PinHeader_1x04_P2.54mm_Vertical, symbol Connector:Conn_01x04_Female
- added MX1, MX2, MX3, MX4: MX-NoLED, SamacSys_Parts:MXOnly-1U-NoLED_3Pins, symbol MX_Alps_Hybrid:MX-NoLED
- added U1: IS31FL3741-QFLS4-TR, Breadboard:IS31FL3741-QFLS4-TR, symbol Breadbord:IS31FL3741-QFLS4-TR
- J17: footprint SamacSys_Parts:SWR204NRTND03STGA -> Connector_PinHeader_2.54mm:PinHeader_2x03_P2.54mm_Vertical
Connections:
- net at J14.1 (Pin_1): now also IC3.33 (PE0_[~{WR]})
- net at J14.10 (Pin_10): now also IC3.42 (PC7_[A15/IC.3/CLKO])
- net at J14.11 (Pin_11): now also IC3.43 (PE2_[ALE/~{HWB]})
- net at J14.12 (Pin_12): now also IC3.44 (PA7_[AD7])
- net at J14.13 (Pin_13): now also IC3.45 (PA6_[AD6])
- net at J14.14 (Pin_14): now also IC3.46 (PA5_[AD5])
- net at J14.15 (Pin_15): now also IC3.47 (PA4_[AD4])
- net at J14.16 (Pin_16): now also IC3.48 (PA3_[AD3])
- net at J14.17 (Pin_17): now also IC3.49 (PA2_[AD2])
- net at J14.18 (Pin_18): now also IC3.50 (PA1_[AD1])
- net at J14.19 (Pin_19): now also IC3.51 (PA0_[AD0])
- net at J14.2 (Pin_2): now also IC3.34 (PE1_[~{RD]})
- net at J14.20 (Pin_20): now also IC3.52 (VCC_1)
- net GND_1: now reaches J14.21 (Pin_21)
- net GND_1: now also J13.22 (Pin_22), J14.31 (Pin_31), IC3.22 (GND), IC3.53 (GND_1), IC3.63 (GND_2)
- net at J14.22 (Pin_22): now also IC3.54 (PF7_[ADC7/TDI])
- net at J14.23 (Pin_23): now also IC3.55 (PF6_[ADC6/TDO])
- net at J14.24 (Pin_24): now also IC3.56 (PF5_[ADC5/TMS])
- net at J14.25 (Pin_25): now also IC3.57 (PF4_[ADC4/TCK])
- net at J14.26 (Pin_26): now also IC3.58 (PF3_[ADC3])
- net at J14.27 (Pin_27): now also IC3.59 (PF2_[ADC2])
- net at J14.28 (Pin_28): now also IC3.60 (PF1_[ADC1])
- net at J14.29 (Pin_29): now also IC3.61 (PF0_[ADC0])
- net at J14.3 (Pin_3): now also IC3.35 (PC0_[A8])
- net at J14.30 (Pin_30): now also IC3.62 (AREF)
- net at J14.32 (Pin_32): now also IC3.64 (AVCC)
- net at J14.4 (Pin_4): now also IC3.36 (PC1_[A9])
- net at J14.5 (Pin_5): now also IC3.37 (PC2_[A10])
- net at J14.6 (Pin_6): now also IC3.38 (PC3_[A11/T.3])
- net at J14.7 (Pin_7): now also IC3.39 (PC4_[A12/OC.3C])
- net at J14.8 (Pin_8): now also IC3.40 (PC5_[A13/OC.3B])
- net at J14.9 (Pin_9): now also IC3.41 (PC6_[A14/OC.3A])
- net GND_5: now reaches J19.1 (Pin_1), U2.1 (GND)
- net GND_2: now reaches J16.5 (Pin_5), USB1.12 (GND)
- net GND_2: now also J15.1 (Pin_1), USB1.1 (GND)
- net at J13.1 (Pin_1): now also IC3.1 ([INT.6/AIN.0]_PE6)
- net at J13.10 (Pin_10): now also IC3.10 ([SS/PCINT0]_PB0)
- net at J13.11 (Pin_11): now also IC3.11 ([PCINT1/SCLK]_PB1)
- net at J13.12 (Pin_12): now also IC3.12 ([PDI/PCINT2/MOSI]_PB2)
- net at J13.13 (Pin_13): now also IC3.13 ([PDO/PCINT3/MISO]_PB3)
- net at J13.14 (Pin_14): now also IC3.14 ([PCINT4/OC.2A]_PB4)
- net at J13.15 (Pin_15): now also IC3.15 ([PCINT5/OC.1A]_PB5)
- net at J13.16 (Pin_16): now also IC3.16 ([PCINT6/OC.1B]_PB6)
- net at J13.17 (Pin_17): now also IC3.17 ([PCINT7/OC.0A/OC.1C]_PB7)
- net at J13.18 (Pin_18): now also IC3.18 ([INT4/TOSC1]_PE4)
- net at J13.19 (Pin_19): now also IC3.19 ([INT.5/TOSC2]_PE5)
- net at J13.2 (Pin_2): now also IC3.2 ([INT.7/AIN.1/UVCON]_PE7)
- net at J13.20 (Pin_20): now also IC3.20 (~{RESET})
- net at J13.21 (Pin_21): now also IC3.21 (VCC)
- net at J13.23 (Pin_23): now also IC3.23 (XTAL2)
- net at J13.24 (Pin_24): now also IC3.24 (XTAL1)
- net at J13.25 (Pin_25): now also IC3.25 ([OC0B/SCL/INT0]_PD0)
- net at J13.26 (Pin_26): now also IC3.26 ([OC2B/SDA/INT1]_PD1)
- net at J13.27 (Pin_27): now also IC3.27 ([RXD1/INT2]_PD2)
- net at J13.28 (Pin_28): now also IC3.28 ([TXD1/INT3]_PD3)
- net at J13.29 (Pin_29): now also IC3.29 ([ICP1]_PD4)
- net at J13.3 (Pin_3): now also IC3.3 (UVCC)
- net at J13.30 (Pin_30): now also IC3.30 ([XCK1]_PD5)
- net at J13.31 (Pin_31): now also IC3.31 ([T1]_PD6)
- net at J13.32 (Pin_32): now also IC3.32 ([T0]_PD7)
- net at J13.4 (Pin_4): now also IC3.4 (D-)
- net at J13.5 (Pin_5): now also IC3.5 (D+)
- net at J13.6 (Pin_6): now also IC3.6 (UGND)
- net at J13.7 (Pin_7): now also IC3.7 (UCAP)
- net at J13.8 (Pin_8): now also IC3.8 (VBUS)
- net at J13.9 (Pin_9): now also IC3.9 ([IUID]_PE3)
- net at J3.1 (Pin_1): now also U1.1 (CS34)
- net at J3.10 (Pin_10): now also U1.10 (SCL)
- net at J3.11 (Pin_11): now also U1.11 (SDB)
- net GND_3: now reaches J3.12 (Pin_12)
- net GND_3: now also J4.25 (Pin_25), J4.6 (Pin_6), U1.12 (GND), U1.36 (GND), U1.55 (GND), U1.61 (GND)
- net at J3.13 (Pin_13): now also U1.13 (R_EXT)
- net at J3.14 (Pin_14): now also U1.14 (AVCC)
- net at J3.15 (Pin_15): now also U1.15 (PVCC)
- net at J3.16 (Pin_16): now also U1.16 (SW1)
- net at J3.17 (Pin_17): now also U1.17 (SW2)
- net at J3.18 (Pin_18): now also U1.18 (SW3)
- net at J3.19 (Pin_19): now also U1.19 (SW4)
- net at J3.2 (Pin_2): now also U1.2 (CS35)
- net at J3.20 (Pin_20): now also U1.20 (SW5)
- net at J3.21 (Pin_21): now also U1.21 (SW6)
- net at J3.22 (Pin_22): now also U1.22 (SW7)
- net at J3.23 (Pin_23): now also U1.23 (SW8)
- net at J3.24 (Pin_24): now also U1.24 (SW9)
- net at J3.25 (Pin_25): now also U1.25 (PVCC)
- net at J3.26 (Pin_26): now also U1.26 (CS1)
- net at J3.27 (Pin_27): now also U1.27 (CS2)
- net at J3.28 (Pin_28): now also U1.28 (CS3)
- net at J3.29 (Pin_29): now also U1.29 (CS4)
- net at J3.3 (Pin_3): now also U1.3 (CS36)
- net at J3.30 (Pin_30): now also U1.30 (CS5)
- net at J4.1 (Pin_1): now also U1.31 (CS6)
- net at J4.2 (Pin_2): now also U1.32 (CS7)
- net at J4.3 (Pin_3): now also U1.33 (CS8)
- net at J4.4 (Pin_4): now also U1.34 (CS9)
- net at J4.5 (Pin_5): now also U1.35 (CS10)
- net at J4.7 (Pin_7): now also U1.37 (CS11)
- net at J4.8 (Pin_8): now also U1.38 (CS12)
- net at J4.9 (Pin_9): now also U1.39 (CS13)
- net at J3.4 (Pin_4): now also U1.4 (CS37)
- net at J4.10 (Pin_10): now also U1.40 (CS14)
- net at J4.11 (Pin_11): now also U1.41 (CS15)
- net at J4.12 (Pin_12): now also U1.42 (CS16)
- net at J4.13 (Pin_13): now also U1.43 (CS17)
- net at J4.14 (Pin_14): now also U1.44 (CS18)
- net at J4.15 (Pin_15): now also U1.45 (CS19)
- net at J4.16 (Pin_16): now also U1.46 (CS20)
- net at J4.17 (Pin_17): now also U1.47 (CS21)
- net at J4.18 (Pin_18): now also U1.48 (CS22)
- net at J4.19 (Pin_19): now also U1.49 (CS23)
- net at J3.5 (Pin_5): now also U1.5 (CS38)
- net at J4.20 (Pin_20): now also U1.50 (CS24)
- net at J4.21 (Pin_21): now also U1.51 (CS25)
- net at J4.22 (Pin_22): now also U1.52 (CS26)
- net at J4.23 (Pin_23): now also U1.53 (CS27)
- net at J4.24 (Pin_24): now also U1.54 (CS28)
- net at J4.26 (Pin_26): now also U1.56 (CS29)
- net at J4.27 (Pin_27): now also U1.57 (CS30)
- net at J4.28 (Pin_28): now also U1.58 (CS31)
- net at J4.29 (Pin_29): now also U1.59 (CS32)
- net at J3.6 (Pin_6): now also U1.6 (CS39)
- net at J4.30 (Pin_30): now also U1.60 (CS33)
- net at J3.7 (Pin_7): now also U1.7 (INTB)
- net at J3.8 (Pin_8): now also U1.8 (ADDR)
- net at J3.9 (Pin_9): now also U1.9 (SDA)
- net GND_7: now reaches J22.1 (Pin_1), U3.1 (NC(GND)@1)
- net GND_7: now also J21.15 (Pin_15), U3.30 (NC(GND)@2)
- net GND_4: now reaches J23.2 (Pin_2), U4.2 (GND)
- net GND_6: now reaches J17.6 (GND), J18.3 (Pin_3)
- new net: J7.3 (Pin_3), MX3.1 (COL)
- new net: J27.3 (Pin_3), MX3.2 (ROW)
- new net: J7.4 (Pin_4), MX4.1 (COL)
- new net: J27.4 (Pin_4), MX4.2 (ROW)
- new net: J7.1 (Pin_1), MX1.1 (COL)
- new net: J27.1 (Pin_1), MX1.2 (ROW)
- new net: J27.2 (Pin_2), MX2.2 (ROW)
- new net: J7.2 (Pin_2), MX2.1 (COL)
Other:
- note added: "Keyboard keys"
- note added: "RGB Leds"
- note added: "Rotary Encoder Switch"
- moved on the sheet: G1, G10, G2, G3, G4, G5, G6, G7, G8, G9, IC1, IC2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

Commit message: Mouse Bits Finished
Connections:
- no-connect marks 0 -> 1
Changed lines of the file:
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@@
   (junction (at 345.44 153.67) (diameter 0) (color 0 0 0 0)
   )
+  (no_connect (at 35.56 226.06))
   (wire (pts (xy 276.86 226.06) (xy 280.67 226.06))
     (stroke (width 0) (type default) (color 0 0 0 0))

Commit message: Updated but something wrong
Parts:
- J1: renamed from J12; value Conn_01x04_Female -> Conn_01x10_Female; footprint Connector_PinHeader_2.54mm:PinHeader_1x04_P2.54mm_Vertical -> Connector_PinHeader_2.54mm:PinHeader_1x10_P2.54mm_Vertical
- J10: renamed from J14; value Conn_01x32_Female -> Conn_01x02_Female; footprint Connector_PinHeader_2.54mm:PinHeader_1x32_P2.54mm_Vertical -> Connector_PinHeader_2.54mm:PinHeader_1x02_P2.54mm_Vertical
- J12: renamed from J13; value Conn_01x32_Female -> Conn_01x02_Female; footprint Connector_PinHeader_2.54mm:PinHeader_1x32_P2.54mm_Vertical -> Connector_PinHeader_2.54mm:PinHeader_1x02_P2.54mm_Vertical
- J13: renamed from J8; value Conn_01x03_Female -> Conn_01x10_Female; footprint Connector_PinHeader_2.54mm:PinHeader_1x03_P2.54mm_Vertical -> Connector_PinHeader_2.54mm:PinHeader_1x10_P2.54mm_Vertical
- J14: renamed from J17; value AVR-ISP-6 -> Conn_01x02_Female; footprint Connector_PinHeader_2.54mm:PinHeader_2x03_P2.54mm_Vertical -> Connector_PinHeader_2.54mm:PinHeader_1x02_P2.54mm_Vertical
- J15: renamed from J18; value Conn_01x03_Female -> Conn_01x02_Female; footprint Connector_PinHeader_2.54mm:PinHeader_1x03_P2.54mm_Vertical -> Connector_PinHeader_2.54mm:PinHeader_1x02_P2.54mm_Vertical
- J18: renamed from J5; value Conn_01x02_Female -> Conn_01x10_Female; footprint Connector_PinHeader_2.54mm:PinHeader_1x02_P2.54mm_Vertical -> Connector_PinHeader_2.54mm:PinHeader_1x10_P2.54mm_Vertical
- J19: renamed from J6; value Conn_01x02_Female -> Conn_01x10_Female; footprint Connector_PinHeader_2.54mm:PinHeader_1x02_P2.54mm_Vertical -> Connector_PinHeader_2.54mm:PinHeader_1x10_P2.54mm_Vertical
- J2: renamed from J11; value Conn_01x06_Female -> Conn_01x10_Female; footprint Connector_PinHeader_2.54mm:PinHeader_1x06_P2.54mm_Vertical -> Connector_PinHeader_2.54mm:PinHeader_1x10_P2.54mm_Vertical
- J20: renamed from J23; value Conn_01x03_Female -> Conn_01x32_Female; footprint Connector_PinHeader_2.54mm:PinHeader_1x03_P2.54mm_Vertical -> Connector_PinHeader_2.54mm:PinHeader_1x32_P2.54mm_Vertical
- J21: renamed from J24; value Conn_01x02_Female -> Conn_01x04_Female; footprint Connector_PinHeader_2.54mm:PinHeader_1x02_P2.54mm_Vertical -> Connector_PinHeader_2.54mm:PinHeader_1x04_P2.54mm_Vertical
- J24: renamed from J25; value Conn_01x02_Female -> Conn_01x04_Female; footprint Connector_PinHeader_2.54mm:PinHeader_1x02_P2.54mm_Vertical -> Connector_PinHeader_2.54mm:PinHeader_1x04_P2.54mm_Vertical
- J25: renamed from J26; value Conn_01x04_Female -> Conn_01x06_Female; footprint Connector_PinHeader_2.54mm:PinHeader_1x04_P2.54mm_Vertical -> Connector_PinHeader_2.54mm:PinHeader_1x06_P2.54mm_Vertical
- J26: renamed from J3; value Conn_01x30_Female -> Conn_01x10_Female; footprint Connector_PinHeader_2.54mm:PinHeader_1x30_P2.54mm_Vertical -> Connector_PinHeader_2.54mm:PinHeader_1x10_P2.54mm_Vertical
- J27: renamed from J4; value Conn_01x30_Female -> Conn_01x10_Female; footprint Connector_PinHeader_2.54mm:PinHeader_1x30_P2.54mm_Vertical -> Connector_PinHeader_2.54mm:PinHeader_1x10_P2.54mm_Vertical
- J3: renamed from J9; value Conn_01x08_Female -> Conn_01x10_Female; footprint Connector_PinHeader_2.54mm:PinHeader_1x08_P2.54mm_Vertical -> Connector_PinHeader_2.54mm:PinHeader_1x10_P2.54mm_Vertical
- J4: renamed from J10; value Conn_01x08_Female -> Conn_01x10_Female; footprint Connector_PinHeader_2.54mm:PinHeader_1x08_P2.54mm_Vertical -> Connector_PinHeader_2.54mm:PinHeader_1x10_P2.54mm_Vertical
- J5: renamed from J15; value Conn_01x07_Female -> Conn_01x04_Female; footprint Connector_PinHeader_2.54mm:PinHeader_1x07_P2.54mm_Vertical -> Connector_PinHeader_2.54mm:PinHeader_1x04_P2.54mm_Vertical
- J6: renamed from J16; value Conn_01x07_Female -> Conn_01x03_Female; footprint Connector_PinHeader_2.54mm:PinHeader_1x07_P2.54mm_Vertical -> Connector_PinHeader_2.54mm:PinHeader_1x03_P2.54mm_Vertical
- J9: renamed from J7; value Conn_01x04_Female -> Conn_01x10_Female; footprint Connector_PinHeader_2.54mm:PinHeader_1x04_P2.54mm_Vertical -> Connector_PinHeader_2.54mm:PinHeader_1x10_P2.54mm_Vertical
- U1: renamed from U2; value PRTR5V0U2X -> AP2112K-3.3; footprint random-keyboard-parts:SOT143B -> SamacSys_Parts:SOT95P282X130-5N
- U2: renamed from U4; value AP2112K-3.3 -> QFN40P700X700X80-61N-D; footprint SamacSys_Parts:SOT95P282X130-5N -> SamacSys_Parts:QFN40P700X700X80-61N-D
- U3: renamed from U1; value IS31FL3741-QFLS4-TR -> PRTR5V0U2X; footprint Breadboard:IS31FL3741-QFLS4-TR -> random-keyboard-parts:SOT143B
- renumbered IC3 to IC1, IC1 to IC2, IC2 to IC3, J27 to J11, J1 to J16, J2 to J17, J19 to J7, J20 to J8, J22 to JOLED1, J21 to JOLED2, U3 to UOLED1
