File: ProtoFull/ProtoFull.kicad_sch (KiCad schematic)
At the start: 0 parts

Commit message: Updates on the schematics
Parts:
- added C? (x3): 1uF, 0603-NO, symbol Adafruit IS31FL3741 Matrix-eagle-import:CAP_CERAMIC0603_NO
- added C? (x3): 0.1uF, Capacitor_SMD:C_0805_2012Metric, symbol Device:C_Small
- added C? (x4): 10uF, 0805-NO, symbol Adafruit IS31FL3741 Matrix-eagle-import:CAP_CERAMIC0805-NOOUTLINE
- added C? (x5): 10uF, 0805-NO, symbol Adafruit 1.3in 128x64 OLED STEMMA QT-eagle-import:CAP_CERAMIC0805-NOOUTLINE
- added C? (x2): 22pF, Capacitor_SMD:C_0805_2012Metric, symbol Device:C_Small
- added C?: 1uF, Capacitor_SMD:C_0805_2012Metric, symbol Device:C_Small
- added C? (x2): 2.2uF, 0805-NO, symbol Adafruit 1.3in 128x64 OLED STEMMA QT-eagle-import:CAP_CERAMIC0805-NOOUTLINE
- added C?: 10uF, Capacitor_SMD:C_0805_2012Metric, symbol Device:C_Small
- added C?: 1uF, 0603-NO, symbol Adafruit 1.3in 128x64 OLED STEMMA QT-eagle-import:CAP_CERAMIC0603_NO
- added C?: 0.1uF, 0603-NO, symbol Adafruit 1.3in 128x64 OLED STEMMA QT-eagle-import:CAP_CERAMIC0603_NO
- added D? (x4): LED_BGRA, SamacSys_Parts:QBLP677R-RGB, symbol Device:LED_BGRA
- added D?: GREEN, CHIPLED_0603_NOOUTLINE, symbol Adafruit 1.3in 128x64 OLED STEMMA QT-eagle-import:LED0603_NOOUTLINE
- added D? (x6): SOD-123, Diode_SMD:D_SOD-123, symbol Device:D_Small
- added D?: LED_YELLOW, symbol Device:LED
- added D?: LED_RED, symbol Device:LED
- added F?: 1A, Fuse:Fuse_1206_3216Metric, symbol Device:Polyfuse
- added J?: AVR-ISP-6, SamacSys_Parts:SWR204NRTND03STGA, symbol Connector:AVR-ISP-6
- added MX? (x4): MX-NoLED, SamacSys_Parts:MXOnly-1U-NoLED_3Pins, symbol MX_Alps_Hybrid:MX-NoLED
- added Q? (x2): BSS138, SOT363, symbol Adafruit 1.3in 128x64 OLED STEMMA QT-eagle-import:MOSFET-N_DUAL
- added R? (x2): 10k, Resistor_SMD:R_0805_2012Metric, symbol Device:R_Small
- added R? (x2): 5.1k, Resistor_SMD:R_0805_2012Metric, symbol Device:R_Small
- added R? (x2): 200, Resistor_SMD:R_0805_2012Metric, symbol Device:R_Small
- added R? (x5): 10K, RESPACK_4X0603, symbol Adafruit 1.3in 128x64 OLED STEMMA QT-eagle-import:RESISTOR_4PACK
- added R? (x2): 51, 0603-NO, symbol Adafruit IS31FL3741 Matrix-eagle-import:RESISTOR_0603_NOOUT
- added R? (x2): 22, Resistor_SMD:R_0805_2012Metric, symbol Device:R_Small
- added R? (x2): 4.7K, 0603-NO, symbol Adafruit IS31FL3741 Matrix-eagle-import:RESISTOR_0603_NOOUT
- added R? (x4): 22, 0603-NO, symbol Adafruit IS31FL3741 Matrix-eagle-import:RESISTOR_0603_NOOUT
- added R?: 100K, 0603-NO, symbol Adafruit IS31FL3741 Matrix-eagle-import:RESISTOR_0603_NOOUT
- added R?: 10K, 0603-NO, symbol Adafruit IS31FL3741 Matrix-eagle-import:RESISTOR_0603_NOOUT
- added R?: 390K, 0603-NO, symbol Adafruit 1.3in 128x64 OLED STEMMA QT-eagle-import:RESISTOR_0603_NOOUT
- added R?: 10K, 0603-NO, symbol Adafruit 1.3in 128x64 OLED STEMMA QT-eagle-import:RESISTOR_0603_NOOUT
- added SJ?: SOLDERJUMPER, SOLDERJUMPER_ARROW_NOPASTE, symbol Adafruit 1.3in 128x64 OLED STEMMA QT-eagle-import:SOLDERJUMPER
- added SJ?: SOLDERJUMPERCLOSED, SOLDERJUMPER_CLOSEDWIRE, symbol Adafruit 1.3in 128x64 OLED STEMMA QT-eagle-import:SOLDERJUMPERCLOSED
- added SW? (x2): RotaryEncoder_Switch, symbol Device:RotaryEncoder_Switch
- added SW?: SW_Push, random-keyboard-parts:SKQG-1155865, symbol Switch:SW_Push
- added U?: PRTR5V0U2X, random-keyboard-parts:SOT143B, symbol random-keyboard-parts:PRTR5V0U2X
- added U?: AT90USB1286-AU, SamacSys_Parts:AT90USB1286-AU, symbol MCU_Microchip_AVR:AT90USB1286-AU
- added U?: UG-2864HSWEG01, UG-2864HSWEG01_1.3_WRAPAROUND, symbol Adafruit 1.3in 128x64 OLED STEMMA QT-eagle-import:DISP_OLED_UG-2864HSWEG01
- added U?: AP2112K-3.3, SOT23-5, symbol Adafruit 1.3in 128x64 OLED STEMMA QT-eagle-import:VREG_SOT23-5
- added USB?: HRO-TYPE-C-31-M-12, Type-C:HRO-TYPE-C-31-M-12, symbol Type-C:HRO-TYPE-C-31-M-12
- added X?: IS31FL3741, QFN60_7MM, symbol Adafruit IS31FL3741 Matrix-eagle-import:IS31FL3741
- added Y?: 16MHz, Crystal:Crystal_SMD_3225-4Pin_3.2x2.5mm, symbol Device:Crystal_GND24_Small
Connections:
- new net: C?.2, R?.1
- new net: R?.2, USB?.4 (CC1)
- new net: D?.2 (A), MX?.2 (ROW) (x4)
- new net: D?.2 (A), R?.1 (x2)
- new net: C?.2, U?.27 (VCOMH)
- new net: R?.2, U?.2 (IO1), USB?.6 (DP1), USB?.8 (DP2)
- new net: R?.2, U?.3 (IO2), USB?.5 (DN2), USB?.7 (DN1)
- new net: D?.C, R?.1
- new net: R?.2, X?.11 (SDB)
- new net: R?.2, X?.13 (R_EXT)
- new net: R?.1, X?.26 (CS1)
- new net: R?.1, X?.27 (CS2)
- new net: R?.1, X?.28 (CS3)
- new net: R?.1, X?.29 (CS4)
- new net: R?.1, X?.30 (CS5)
- new net: R?.1, X?.31 (CS6)
- new net: C?.1, U?.7 (UCAP)
- new net: R?.1, U?.43 (PE2/~{HWB})
- new net: C?.1, U?.5 (C1N)
- new net: C?.2, U?.4 (C1P)
- new net: D?.2 (A), SW?.S2 (x2)
- new net: R?.2, USB?.10 (CC2)
- new net: C?.1, U?.3 (C2N)
- new net: C?.2, U?.2 (C2P)
- new net: SJ?.2, U?.20 (D2/I2C_SDA)
- new net: R?.2, U?.26 (IREF)
- new net: C?.2, U?.28 (VCC)
- new net +5V: C?.1, C?.2, C?.2, C?.2, C?.2, F?.1, J?.2 (VCC), R?.1, R?.1, R?.2, R?.3 (1), U?.1 (IN), U?.21 (VCC), U?.3 (EN), U?.3 (UVCC), U?.52 (VCC), U?.64 (AVCC), U?.8 (VBUS)
- new net 3.3V: C?.1, C?.1, C?.2, C?.2, D?.A, Q?.2 (G), Q?.5 (G), R?.2 (1), R?.4 (1), R?.8 (2), U?.11 (BS1), U?.5 (OUT), U?.6 (VBAT), U?.9 (VDD)
- new net COL00: MX?.1 (COL), MX?.1 (COL), U?.35 (PC0)
- new net COL01: MX?.1 (COL), MX?.1 (COL), U?.36 (PC1)
- new net COL02: SW?.S1, SW?.S1, U?.37 (PC2)
- new net CS1_B: D?.1 (BK), D?.1 (BK), R?.2
- new net CS2_G: D?.2 (GK), D?.2 (GK), R?.2
- new net CS3_R: D?.3 (RK), D?.3 (RK), R?.2
- new net CS4_B: D?.1 (BK), D?.1 (BK), R?.2
- new net CS5_G: D?.2 (GK), D?.2 (GK), R?.2
- new net CS6_R: D?.3 (RK), D?.3 (RK), R?.2
- new net D+: R?.1, U?.5 (D+)
- new net D-: R?.1, U?.4 (D-)
- new net DC/SA0_3.3V: SJ?.2, U?.15 (DC/I2C_SA0)
- new net ENCODER_A1: SW?.A, U?.61 (PF0)
- new net ENCODER_A2: SW?.A, U?.59 (PF2)
- new net ENCODER_B1: SW?.B, U?.60 (PF1)
- new net ENCODER_B2: SW?.B, U?.58 (PF3)
- new net GND: C?.1, C?.1, C?.1, C?.1, C?.1, C?.1, C?.1, C?.1, C?.1, C?.1, C?.2, C?.2, C?.2, C?.2, C?.2, C?.2, C?.2, C?.2, C?.2, C?.2, D?.1 (K), D?.1 (K), J?.6 (GND), R?.1, R?.1, R?.1, R?.1, R?.1, R?.2, R?.2, SJ?.1, SW?.1, SW?.C, SW?.C, U?.1 (GND), U?.1 (NC(GND)@1), U?.10 (BS0), U?.12 (BS2), U?.2 (GND), U?.22 (GND), U?.29 (VLSS), U?.30 (NC(GND)@2), U?.53 (GND), U?.6 (UGND), U?.63 (GND), U?.8 (VSS), USB?.1 (GND), USB?.12 (GND), USB?.13 (SHIELD), X?.12 (GND), X?.36 (GND), X?.55 (GND), X?.8 (ADDR), X?.THERMAL (GND), Y?.2, Y?.4
- new net MISO: J?.1 (MISO), U?.13 (PB3)
- new net MOSI: J?.4 (MOSI), U?.12 (PB2)
- new net RESET: J?.5 (~{RST}), R?.2, SW?.2, U?.14 (/RES), U?.20 (~{RESET})
- new net ROT1_ROW: D?.1 (K), D?.1 (K), D?.1 (K), U?.34 (PE1)
- new net ROT2_ROW: D?.1 (K), D?.1 (K), D?.1 (K), U?.33 (PE0)
- new net SCK: J?.3 (SCK), U?.11 (PB1)
- new net SCL: Q?.6 (D), R?.1, R?.8 (2), U?.25 (PD0), X?.10 (SCL)
- new net SCL_3.3: Q?.1 (S), R?.7 (2), U?.18 (D0/SPI_SCLK/I2C_SCK)
- new net SDA: Q?.3 (D), R?.1, R?.6 (2), U?.26 (PD1), X?.9 (SDA)
- new net SDA_3.3: Q?.4 (S), R?.5 (2), SJ?.1, U?.19 (D1/SPI_SDIN/I2C_SDA)
- new net SW1: D?.4 (A), D?.4 (A), X?.16 (SW1)
- new net SW2: D?.4 (A), D?.4 (A), X?.17 (SW2)
- new net VCC: C?.1, C?.1, C?.1, C?.1, C?.1, C?.1, C?.1, F?.2, R?.2, R?.2, R?.2, U?.4 (VCC), USB?.11 (VBUS), USB?.2 (VBUS), X?.14 (AVCC), X?.15 (PVCC), X?.25 (PVCC)
- new net XTAL1: C?.2, U?.24 (XTAL1), Y?.1
- new net XTAL2: C?.2, U?.23 (XTAL2), Y?.3
- no-connect marks 0 -> 37
Other:
- note added: "30 Pins Oled Connector"
- note added: "Connector Header Right Angle 6 position 2.00mm"
- note added: "Crystal"
- note added: "D"
- note added: "Fuse"
- note added: "G"
- note added: "I2C"
- note added: "I2C Pullups & Shift"
- note added: "Keyboard keys"
- note added: "Keyboard keys LED"
- note added: "MCU"
- note added: "MCU Decoplings"
- note added: "Master Led Driver"
- note added: "ON LED"
- note added: "Open for"
- note added: "Power supply"
- note added: "Rotary Encoders"
- note added: "S"
- note added: "USB Type-C"

Commit message: Breadboad
Parts:
- C10, C17, C21, C3, C8: renamed from C?; footprint 0603-NO -> Capacitor_SMD:C_0805_2012Metric
- C15, C16, C18, C19, C20, C22, C23, C5, C6, C7, C9: renamed from C?; footprint 0805-NO -> Capacitor_SMD:C_0805_2012Metric
- R10, R11, R12, R13, R14, R15, R16, R17, R21, R22, R8, R9: renamed from R?; footprint 0603-NO -> Resistor_SMD:R_0805_2012Metric
- R19, R20: renamed from R?; footprint RESPACK_4X0603 -> Resistor_SMD:R_0805_2012Metric
- gave numbers to parts that had none: 47

Commit message: Panel Gerber and Internet Shortcuts for proto
Parts:
- D13: footprint CHIPLED_0603_NOOUTLINE -> (none)
- Q1: footprint SOT363 -> (none)
- SJ1: footprint SOLDERJUMPER_ARROW_NOPASTE -> (none)
- SJ2: footprint SOLDERJUMPER_CLOSEDWIRE -> (none)
- U3: footprint UG-2864HSWEG01_1.3_WRAPAROUND -> (none)
- U4: footprint SOT23-5 -> (none)
- X1: footprint QFN60_7MM -> (none)
Changed lines of the file:
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@@
     (property "Reference" "D13" (id 0) (at 109.855 358.14 0))
     (property "Value" "GREEN" (id 1) (at 102.616 358.14 0))
-    (property "Footprint" "CHIPLED_0603_NOOUTLINE" (id 2) (at 105.41 359.41 0)
+    (property "Footprint" "" (id 2) (at 105.41 359.41 0)
       (effects (font (size 1.27 1.27)) hide)
     )
@@
       (effects (font (size 1.27 1.0795)) (justify left bottom))
     )
-    (property "Footprint" "QFN60_7MM" (id 2) (at 262.89 129.54 0)
+    (property "Footprint" "" (id 2) (at 262.89 129.54 0)
       (effects (font (size 1.27 1.27)) hide)
     )
@@
       (effects (font (size 1.27 1.0795)) (justify left bottom))
     )
-    (property "Footprint" "SOLDERJUMPER_ARROW_NOPASTE" (id 2) (at 266.7 342.9 0)
+    (property "Footprint" "" (id 2) (at 266.7 342.9 0)
       (effects (font (size 1.27 1.27)) hide)
     )
@@
       (effects (font (size 1.27 1.0795)) (justify left bottom))
     )
-    (property "Footprint" "SOT363" (id 2) (at 177.8 361.95 0)
+    (property "Footprint" "" (id 2) (at 177.8 361.95 0)
       (effects (font (size 1.27 1.27)) hide)
     )
@@
       (effects (font (size 1.27 1.27)) (justify left bottom))
     )
-    (property "Footprint" "UG-2864HSWEG01_1.3_WRAPAROUND" (id 2) (at 322.58 337.82 0)
+    (property "Footprint" "" (id 2) (at 322.58 337.82 0)
       (effects (font (size 1.27 1.27)) hide)
     )
@@
       (effects (font (size 1.27 1.0795)) (justify left bottom))
     )
-    (property "Footprint" "SOT363" (id 2) (at 167.64 372.11 0)
+    (property "Footprint" "" (id 2) (at 167.64 372.11 0)
       (effects (font (size 1.27 1.27)) hide)
     )
@@
       (effects (font (size 1.27 1.0795)) (justify left bottom))
     )
-    (property "Footprint" "SOT23-5" (id 2) (at 57.15 356.87 0)
+    (property "Footprint" "" (id 2) (at 57.15 356.87 0)
       (effects (font (size 1.27 1.27)) hide)
     )
@@
       (effects (font (size 1.27 1.0795)) (justify left bottom))
     )
-    (property "Footprint" "SOLDERJUMPER_CLOSEDWIRE" (id 2) (at 287.02 353.06 0)
+    (property "Footprint" "" (id 2) (at 287.02 353.06 0)
       (effects (font (size 1.27 1.27)) hide)
     )
@@
     )
     (path "/3be384a3-611a-4689-8b31-165c4fb97bc9"
-      (reference "D13") (unit 1) (value "GREEN") (footprint "CHIPLED_0603_NOOUTLINE")
+      (reference "D13") (unit 1) (value "GREEN") (footprint "")
     )
     (path "/c1b5c04b-ab1a-4fda-a1fc-51b5d0513ce4"
@@
     )
     (path "/c9db1c7a-6507-4d61-b504-2d7dc9e8f7de"
-      (reference "Q1") (unit 1) (value "BSS138") (footprint "SOT363")
+      (reference "Q1") (unit 1) (value "BSS138") (footprint "")
     )
     (path "/ac3fdcbb-4c48-4df8-b03e-fefd52c64a65"
-      (reference "Q1") (unit 2) (value "BSS138") (footprint "SOT363")
+      (reference "Q1") (unit 2) (value "BSS138") (footprint "")
     )
     (path "/246d4f1e-d0c8-4322-8e19-fc45f445ab98"
@@
     )
     (path "/431c1da1-02e7-418b-86af-e03aec778d3e"
-      (reference "SJ1") (unit 1) (value "SOLDERJUMPER") (footprint "SOLDERJUMPER_ARROW_NOPASTE")
+      (reference "SJ1") (unit 1) (value "SOLDERJUMPER") (footprint "")
     )
     (path "/f2271207-6fd1-4c24-99f5-29a1f078a658"
-      (reference "SJ2") (unit 1) (value "SOLDERJUMPERCLOSED") (footprint "SOLDERJUMPER_CLOSEDWIRE")
+      (reference "SJ2") (unit 1) (value "SOLDERJUMPERCLOSED") (footprint "")
     )
     (path "/bf788b48-e4d3-4e3f-a55a-e725955e8659"
@@
     )
     (path "/c8640ec3-d706-41e6-8319-0ce72026615c"
-      (reference "U3") (unit 1) (value "UG-2864HSWEG01") (footprint "UG-2864HSWEG01_1.3_WRAPAROUND")
+      (reference "U3") (unit 1) (value "UG-2864HSWEG01") (footprint "")
     )
     (path "/f0fcc5f6-1571-4c72-b648-71bdb560be87"
-      (reference "U4") (unit 1) (value "AP2112K-3.3") (footprint "SOT23-5")
+      (reference "U4") (unit 1) (value "AP2112K-3.3") (footprint "")
     )
     (path "/976416f1-f46a-461b-8803-72085c8434d4"
@@
     )
     (path "/403ba84f-94b3-4488-8350-ec0ce6e87e0b"
-      (reference "X1") (unit 1) (value "IS31FL3741") (footprint "QFN60_7MM")
+      (reference "X1") (unit 1) (value "IS31FL3741") (footprint "")
     )
     (path "/47876792-b1d9-4826-b4a3-ca899dd41374"

Commit message: Small alignment error for the crystal in the panel
Parts:
- D1, D12, D13: footprint (none) -> LED_SMD:LED_0805_2012Metric
- Q1: footprint (none) -> SamacSys_Parts:SOT95P240X120-3N
- SJ1, SJ2: footprint (none) -> random-keyboard-parts:Jumper-UserFriendly
- SW2, SW3: footprint (none) -> Rotary_Encoder:RotaryEncoder_Alps_EC12E_Vertical_H20mm
- U3: footprint (none) -> SamacSys_Parts:5051103091
- U4: footprint (none) -> Package_TO_SOT_SMD:SOT-223-3_TabPin2
- X1: footprint (none) -> Breadboard:IS31FL3741-QFLS4-TR
Changed lines of the file:
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@@
     (property "Reference" "D13" (id 0) (at 109.855 358.14 0))
     (property "Value" "GREEN" (id 1) (at 102.616 358.14 0))
-    (property "Footprint" "" (id 2) (at 105.41 359.41 0)
+    (property "Footprint" "LED_SMD:LED_0805_2012Metric" (id 2) (at 105.41 359.41 0)
       (effects (font (size 1.27 1.27)) hide)
     )
@@
       (effects (font (size 1.27 1.0795)) (justify left bottom))
     )
-    (property "Footprint" "" (id 2) (at 262.89 129.54 0)
+    (property "Footprint" "Breadboard:IS31FL3741-QFLS4-TR" (id 2) (at 262.89 129.54 0)
       (effects (font (size 1.27 1.27)) hide)
     )
@@
       (effects (font (size 1.27 1.0795)) (justify left bottom))
     )
-    (property "Footprint" "" (id 2) (at 266.7 342.9 0)
+    (property "Footprint" "random-keyboard-parts:Jumper-UserFriendly" (id 2) (at 266.7 342.9 0)
       (effects (font (size 1.27 1.27)) hide)
     )
@@
     (property "Reference" "D12" (id 0) (at 146.3675 131.0345 0))
     (property "Value" "LED_YELLOW" (id 1) (at 146.3675 133.8096 0))
-    (property "Footprint" "" (id 2) (at 144.78 137.16 0)
+    (property "Footprint" "LED_SMD:LED_0805_2012Metric" (id 2) (at 144.78 137.16 0)
       (effects (font (size 1.27 1.27)) hide)
     )
@@
     (property "Reference" "D1" (id 0) (at 150.1775 19.2745 0))
     (property "Value" "LED_RED" (id 1) (at 150.1775 22.0496 0))
-    (property "Footprint" "" (id 2) (at 148.59 25.4 0)
+    (property "Footprint" "LED_SMD:LED_0805_2012Metric" (id 2) (at 148.59 25.4 0)
       (effects (font (size 1.27 1.27)) hide)
     )
@@
       (effects (font (size 1.27 1.27)) (justify right))
     )
-    (property "Footprint" "" (id 2) (at 191.516 46.99 0)
+    (property "Footprint" "Rotary_Encoder:RotaryEncoder_Alps_EC12E_Vertical_H20mm" (id 2) (at 191.516 46.99 0)
       (effects (font (size 1.27 1.27)) hide)
     )
@@
       (effects (font (size 1.27 1.0795)) (justify left bottom))
     )
-    (property "Footprint" "" (id 2) (at 177.8 361.95 0)
+    (property "Footprint" "SamacSys_Parts:SOT95P240X120-3N" (id 2) (at 177.8 361.95 0)
       (effects (font (size 1.27 1.27)) hide)
     )
@@
       (effects (font (size 1.27 1.27)) (justify left bottom))
     )
-    (property "Footprint" "" (id 2) (at 322.58 337.82 0)
+    (property "Footprint" "SamacSys_Parts:5051103091" (id 2) (at 322.58 337.82 0)
       (effects (font (size 1.27 1.27)) hide)
     )
@@
       (effects (font (size 1.27 1.0795)) (justify left bottom))
     )
-    (property "Footprint" "" (id 2) (at 167.64 372.11 0)
+    (property "Footprint" "SamacSys_Parts:SOT95P240X120-3N" (id 2) (at 167.64 372.11 0)
       (effects (font (size 1.27 1.27)) hide)
     )
@@
       (effects (font (size 1.27 1.27)) (justify right))
     )
-    (property "Footprint" "" (id 2) (at 237.236 46.99 0)
+    (property "Footprint" "Rotary_Encoder:RotaryEncoder_Alps_EC12E_Vertical_H20mm" (id 2) (at 237.236 46.99 0)
       (effects (font (size 1.27 1.27)) hide)
     )
@@
       (effects (font (size 1.27 1.0795)) (justify left bottom))
     )
-    (property "Footprint" "" (id 2) (at 57.15 356.87 0)
+    (property "Footprint" "Package_TO_SOT_SMD:SOT-223-3_TabPin2" (id 2) (at 57.15 356.87 0)
       (effects (font (size 1.27 1.27)) hide)
     )
@@
       (effects (font (size 1.27 1.0795)) (justify left bottom))
     )
-    (property "Footprint" "" (id 2) (at 287.02 353.06 0)
+    (property "Footprint" "random-keyboard-parts:Jumper-UserFriendly" (id 2) (at 287.02 353.06 0)
       (effects (font (size 1.27 1.27)) hide)
     )
@@
     )
     (path "/9ce7cc78-97a9-4666-8f05-2cea2c76ae51"
-      (reference "D1") (unit 1) (value "LED_RED") (footprint "")
+      (reference "D1") (unit 1) (value "LED_RED") (footprint "LED_SMD:LED_0805_2012Metric")
     )
     (path "/d8fc968d-0334-4506-9468-5085bda493cb"
@@
     )
     (path "/4ae97565-2708-4414-9613-e95d09635fba"
-      (reference "D12") (unit 1) (value "LED_YELLOW") (footprint "")
+      (reference "D12") (unit 1) (value "LED_YELLOW") (footprint "LED_SMD:LED_0805_2012Metric")
     )
     (path "/3be384a3-611a-4689-8b31-165c4fb97bc9"
-      (reference "D13") (unit 1) (value "GREEN") (footprint "")
+      (reference "D13") (unit 1) (value "GREEN") (footprint "LED_SMD:LED_0805_2012Metric")
     )
     (path "/c1b5c04b-ab1a-4fda-a1fc-51b5d0513ce4"
@@
     )
     (path "/c9db1c7a-6507-4d61-b504-2d7dc9e8f7de"
-      (reference "Q1") (unit 1) (value "BSS138") (footprint "")
+      (reference "Q1") (unit 1) (value "BSS138") (footprint "SamacSys_Parts:SOT95P240X120-3N")
     )
     (path "/ac3fdcbb-4c48-4df8-b03e-fefd52c64a65"
-      (reference "Q1") (unit 2) (value "BSS138") (footprint "")
+      (reference "Q1") (unit 2) (value "BSS138") (footprint "SamacSys_Parts:SOT95P240X120-3N")
     )
     (path "/246d4f1e-d0c8-4322-8e19-fc45f445ab98"
@@
     )
     (path "/431c1da1-02e7-418b-86af-e03aec778d3e"
-      (reference "SJ1") (unit 1) (value "SOLDERJUMPER") (footprint "")
+      (reference "SJ1") (unit 1) (value "SOLDERJUMPER") (footprint "random-keyboard-parts:Jumper-UserFriendly")
     )
     (path "/f2271207-6fd1-4c24-99f5-29a1f078a658"
-      (reference "SJ2") (unit 1) (value "SOLDERJUMPERCLOSED") (footprint "")
+      (reference "SJ2") (unit 1) (value "SOLDERJUMPERCLOSED") (footprint "random-keyboard-parts:Jumper-UserFriendly")
     )
     (path "/bf788b48-e4d3-4e3f-a55a-e725955e8659"
@@
     )
     (path "/9dc96a6a-c0a1-49cb-8839-0153da4f7d99"
-      (reference "SW2") (unit 1) (value "RotaryEncoder_Switch") (footprint "")
+      (reference "SW2") (unit 1) (value "RotaryEncoder_Switch") (footprint "Rotary_Encoder:RotaryEncoder_Alps_EC12E_Vertical_H20mm")
     )
     (path "/e60dee01-ae30-422b-b4f0-b09b086d7dae"
-      (reference "SW3") (unit 1) (value "RotaryEncoder_Switch") (footprint "")
+      (reference "SW3") (unit 1) (value "RotaryEncoder_Switch") (footprint "Rotary_Encoder:RotaryEncoder_Alps_EC12E_Vertical_H20mm")
     )
     (path "/36602f07-d10c-4d2e-a6d7-b32030e0d118"
@@
     )
     (path "/c8640ec3-d706-41e6-8319-0ce72026615c"
-      (reference "U3") (unit 1) (value "UG-2864HSWEG01") (footprint "")
+      (reference "U3") (unit 1) (value "UG-2864HSWEG01") (footprint "SamacSys_Parts:5051103091")
     )
     (path "/f0fcc5f6-1571-4c72-b648-71bdb560be87"
-      (reference "U4") (unit 1) (value "AP2112K-3.3") (footprint "")
+      (reference "U4") (unit 1) (value "AP2112K-3.3") (footprint "Package_TO_SOT_SMD:SOT-223-3_TabPin2")
     )
     (path "/976416f1-f46a-461b-8803-72085c8434d4"
@@
     )
     (path "/403ba84f-94b3-4488-8350-ec0ce6e87e0b"
-      (reference "X1") (unit 1) (value "IS31FL3741") (footprint "")
+      (reference "X1") (unit 1) (value "IS31FL3741") (footprint "Breadboard:IS31FL3741-QFLS4-TR")
     )
     (path "/47876792-b1d9-4826-b4a3-ca899dd41374"
