File: ProtoFull/ProtoFull.kicad_sch (KiCad schematic)
At the start: 77 parts, among them J1 AVR-ISP-6, Q1 BSS138, SW1 SW_Push, SW2 RotaryEncoder_Switch, SW3 RotaryEncoder_Switch, U1 PRTR5V0U2X, U2 AT90USB1286-AU, U3 UG-2864HSWEG01, U4 AP2112K-3.3, X1 IS31FL3741, Y1 16MHz

Commit message: Merge Schematics, OLED not sure
Parts:
- removed C1: 1uF, Capacitor_SMD:C_0805_2012Metric, symbol Device:C_Small
- removed C10, C3, C8: 1uF, Capacitor_SMD:C_0805_2012Metric, symbol Adafruit IS31FL3741 Matrix-eagle-import:CAP_CERAMIC0603_NO
- removed C11: 10uF, Capacitor_SMD:C_0805_2012Metric, symbol Device:C_Small
- removed C12, C13, C14: 0.1uF, Capacitor_SMD:C_0805_2012Metric, symbol Device:C_Small
- removed C15, C16: 2.2uF, Capacitor_SMD:C_0805_2012Metric, symbol Adafruit 1.3in 128x64 OLED STEMMA QT-eagle-import:CAP_CERAMIC0805-NOOUTLINE
- removed C17: 1uF, Capacitor_SMD:C_0805_2012Metric, symbol Adafruit 1.3in 128x64 OLED STEMMA QT-eagle-import:CAP_CERAMIC0603_NO
- removed C18, C19, C20, C22, C23: 10uF, Capacitor_SMD:C_0805_2012Metric, symbol Adafruit 1.3in 128x64 OLED STEMMA QT-eagle-import:CAP_CERAMIC0805-NOOUTLINE
- removed C2, C4: 22pF, Capacitor_SMD:C_0805_2012Metric, symbol Device:C_Small
- removed C21: 0.1uF, Capacitor_SMD:C_0805_2012Metric, symbol Adafruit 1.3in 128x64 OLED STEMMA QT-eagle-import:CAP_CERAMIC0603_NO
- removed C5, C6, C7, C9: 10uF, Capacitor_SMD:C_0805_2012Metric, symbol Adafruit IS31FL3741 Matrix-eagle-import:CAP_CERAMIC0805-NOOUTLINE
- removed D12: LED_YELLOW, LED_SMD:LED_0805_2012Metric, symbol Device:LED
- removed D13: GREEN, LED_SMD:LED_0805_2012Metric, symbol Adafruit 1.3in 128x64 OLED STEMMA QT-eagle-import:LED0603_NOOUTLINE
- removed D2, D3, D6, D7, D8, D9: SOD-123, Diode_SMD:D_SOD-123, symbol Device:D_Small
- removed D4, D5: LED_BGRA, SamacSys_Parts:QBLP677R-RGB, symbol Device:LED_BGRA
- removed Q1: BSS138, SamacSys_Parts:SOT95P240X120-3N, symbol Adafruit 1.3in 128x64 OLED STEMMA QT-eagle-import:MOSFET-N_DUAL
- removed R1, R18: 200, Resistor_SMD:R_0805_2012Metric, symbol Device:R_Small
- removed R10, R11, R13, R14: 22, Resistor_SMD:R_0805_2012Metric, symbol Adafruit IS31FL3741 Matrix-eagle-import:RESISTOR_0603_NOOUT
- removed R12, R15: 51, Resistor_SMD:R_0805_2012Metric, symbol Adafruit IS31FL3741 Matrix-eagle-import:RESISTOR_0603_NOOUT
- removed R16: 100K, Resistor_SMD:R_0805_2012Metric, symbol Adafruit IS31FL3741 Matrix-eagle-import:RESISTOR_0603_NOOUT
- removed R17: 10K, Resistor_SMD:R_0805_2012Metric, symbol Adafruit IS31FL3741 Matrix-eagle-import:RESISTOR_0603_NOOUT
- removed R19, R20: 10K, Resistor_SMD:R_0805_2012Metric, symbol Adafruit 1.3in 128x64 OLED STEMMA QT-eagle-import:RESISTOR_4PACK
- removed R2, R7: 10k, Resistor_SMD:R_0805_2012Metric, symbol Device:R_Small
- removed R21: 390K, Resistor_SMD:R_0805_2012Metric, symbol Adafruit 1.3in 128x64 OLED STEMMA QT-eagle-import:RESISTOR_0603_NOOUT
- removed R22: 10K, Resistor_SMD:R_0805_2012Metric, symbol Adafruit 1.3in 128x64 OLED STEMMA QT-eagle-import:RESISTOR_0603_NOOUT
- removed R3, R4: 22, Resistor_SMD:R_0805_2012Metric, symbol Device:R_Small
- removed R5, R6: 5.1k, Resistor_SMD:R_0805_2012Metric, symbol Device:R_Small
- removed R8, R9: 4.7K, Resistor_SMD:R_0805_2012Metric, symbol Adafruit IS31FL3741 Matrix-eagle-import:RESISTOR_0603_NOOUT
- removed SJ1: SOLDERJUMPER, random-keyboard-parts:Jumper-UserFriendly, symbol Adafruit 1.3in 128x64 OLED STEMMA QT-eagle-import:SOLDERJUMPER
- removed SJ2: SOLDERJUMPERCLOSED, random-keyboard-parts:Jumper-UserFriendly, symbol Adafruit 1.3in 128x64 OLED STEMMA QT-eagle-import:SOLDERJUMPERCLOSED
- removed SW1: SW_Push, random-keyboard-parts:SKQG-1155865, symbol Switch:SW_Push
- removed SW2: RotaryEncoder_Switch, Rotary_Encoder:RotaryEncoder_Alps_EC12E_Vertical_H20mm, symbol Device:RotaryEncoder_Switch
- removed U2: AT90USB1286-AU, SamacSys_Parts:AT90USB1286-AU, symbol MCU_Microchip_AVR:AT90USB1286-AU
- removed U4: AP2112K-3.3, Package_TO_SOT_SMD:SOT-223-3_TabPin2, symbol Adafruit 1.3in 128x64 OLED STEMMA QT-eagle-import:VREG_SOT23-5
- removed USB1: HRO-TYPE-C-31-M-12, Type-C:HRO-TYPE-C-31-M-12, symbol Type-C:HRO-TYPE-C-31-M-12
- removed X1: IS31FL3741, Breadboard:IS31FL3741-QFLS4-TR, symbol Adafruit IS31FL3741 Matrix-eagle-import:IS31FL3741
- removed Y1: 16MHz, Crystal:Crystal_SMD_3225-4Pin_3.2x2.5mm, symbol Device:Crystal_GND24_Small
- added C1, C11, C13, C19: 1uF, Capacitor_SMD:C_0805_2012Metric, symbol Device:C
- added C10, C12, C14, C20, C21, C5, C8, C9: 0.1uF, Capacitor_SMD:C_0805_2012Metric, symbol Device:C
- added C15, C16, C18: 1uF, Capacitor_SMD:C_0805_2012Metric_Pad1.18x1.45mm_HandSolder, symbol Device:C
- added C17: 0.1uF, Capacitor_SMD:C_0805_2012Metric_Pad1.18x1.45mm_HandSolder, symbol Device:C
- added C2, C6: 22pF, Capacitor_SMD:C_0805_2012Metric, symbol Device:C
- added C22: 4,7uF 16V, Capacitor_SMD:C_0805_2012Metric_Pad1.18x1.45mm_HandSolder, symbol Device:C
- added C23: 2,2uF, Capacitor_SMD:C_0805_2012Metric_Pad1.18x1.45mm_HandSolder, symbol Device:C
- added C3, C4, C7: 10uF, Capacitor_SMD:C_0805_2012Metric, symbol Device:C
- added D12, D9: LED_BGRA, SamacSys_Parts:QBLP677R-RGB, symbol Device:LED_BGRA
- added D2, D3, D4, D5, D6, D7: 1N4148W, Diode_SMD:D_SOD-123, symbol Diode:1N4148W
- added D8: GREEN, LED_SMD:LED_0805_2012Metric_Pad1.15x1.40mm_HandSolder, symbol Device:LED
- added IC1: IS31FL3741, SamacSys_Parts:QFN40P700X700X80-61N-D, symbol ProtoFull_Project Libs:IS31FL3741
- added JP1: BS0, ProtoFull_Project Libs:SolderJumper-2_P1.3mm_Open_RoundedPad1.0x1.5mm, symbol Jumper:SolderJumper_2_Open
- added JP2: BS1, ProtoFull_Project Libs:SolderJumper-2_P1.3mm_Open_RoundedPad1.0x1.5mm, symbol Jumper:SolderJumper_2_Bridged
- added JP3: BS2, ProtoFull_Project Libs:SolderJumper-2_P1.3mm_Open_RoundedPad1.0x1.5mm, symbol Jumper:SolderJumper_2_Open
- added JP4: SA0, ProtoFull_Project Libs:SolderJumper-2_P1.3mm_Open_RoundedPad1.0x1.5mm, symbol Jumper:SolderJumper_2_Open
- added JP5: I2C, ProtoFull_Project Libs:SolderJumper-2_P1.3mm_Bridged_RoundedPad1.0x1.5mm, symbol Jumper:SolderJumper_2_Bridged
- added Q1, Q2: BSS138, Package_TO_SOT_SMD:SOT-23, symbol Transistor_FET:BSS138
- added R1: 680, Resistor_SMD:R_0805_2012Metric, symbol Device:R
- added R10, R11, R12, R2, R20, R22, R7, R9: 10k, Resistor_SMD:R_0805_2012Metric, symbol Device:R
- added R13, R14, R16, R17, R3, R4: 22, Resistor_SMD:R_0805_2012Metric, symbol Device:R
- added R15, R18: 51, Resistor_SMD:R_0805_2012Metric, symbol Device:R
- added R19, R21, R23: 10k, Resistor_SMD:R_0805_2012Metric_Pad1.20x1.40mm_HandSolder, symbol Device:R
- added R24: 390k, Resistor_SMD:R_0805_2012Metric_Pad1.20x1.40mm_HandSolder, symbol Device:R
- added R5, R6: 5.1k, Resistor_SMD:R_0805_2012Metric, symbol Device:R
- added R8: 270, Resistor_SMD:R_0805_2012Metric, symbol Device:R
- added SW1: RotaryEncoder_Switch, Rotary_Encoder:RotaryEncoder_Alps_EC12E-Switch_Vertical_H20mm_CircularMountingHoles, symbol Device:RotaryEncoder_Switch
- added SW2: RESET, random-keyboard-parts:PushButton_6x6mm_TH, symbol Switch:SW_Push
- added U2: AT90USB1286-A, Package_QFP:TQFP-64_14x14mm_P0.8mm, symbol MCU_Microchip_AVR:AT90USB1286-A
- added U4: AP2112K-3.3, Package_TO_SOT_SMD:SOT-23-5, symbol Regulator_Linear:AP2112K-3.3
- added USB-C1: HRO-TYPE-C-31-M-12, SamacSys_Parts:TYPE-C-31-M-12, symbol Type-C:HRO-TYPE-C-31-M-12
- added Y1: 16MHz, Crystal:Crystal_SMD_3225-4Pin_3.2x2.5mm_HandSoldering, symbol Device:Crystal_GND24
- D1: footprint LED_SMD:LED_0805_2012Metric -> LED_SMD:LED_0805_2012Metric_Pad1.15x1.40mm_HandSolder
- F1: footprint Fuse:Fuse_1206_3216Metric -> Fuse:Fuse_1206_3216Metric_Pad1.42x1.75mm_HandSolder
- J1: footprint SamacSys_Parts:SWR204NRTND03STGA -> random-keyboard-parts:Reset_Pretty
- MX1, MX2, MX3, MX4: footprint SamacSys_Parts:MXOnly-1U-NoLED_3Pins -> MX_Only:MXOnly-1U-NoLED
- SW3: footprint Rotary_Encoder:RotaryEncoder_Alps_EC12E_Vertical_H20mm -> Rotary_Encoder:RotaryEncoder_Alps_EC12E-Switch_Vertical_H20mm_CircularMountingHoles
- U1: footprint random-keyboard-parts:SOT143B -> Package_TO_SOT_SMD:SOT-143_Handsoldering
Connections:
- net +5V: now also F1.2, C10.1, C11.1, C12.1, C13.1, C14.1, C19.1, C20.1, C3.1, C7.1, C8.1, C9.1, IC1.14 (AVCC), IC1.15 (PVCC), IC1.25 (PVCC), R10.1, R2.1, R20.1, R9.1, U2.21 (VCC), U2.3 (UVCC), U2.52 (VCC), U2.64 (AVCC), U2.8 (VBUS), U4.1 (VIN), U4.3 (EN); no longer F1.1, J1.2 (VCC)
- net COL00: now also U2.35 (PC0)
- net COL01: now also U2.36 (PC1)
- net COL02: now also SW1.S1, U2.37 (PC2)
- net CS1_B: now also D10.1 (BK), D9.1 (BK), R13.2
- net CS2_G: now also D10.2 (GK), D9.2 (GK), R14.2
- net CS3_R: now also D10.3 (RK), D9.3 (RK), R15.2
- net CS4_B: now also D12.1 (BK), R16.2; no longer D10.1 (BK)
- net CS5_G: now also D12.2 (GK), R17.2; no longer D10.2 (GK)
- net CS6_R: now also D12.3 (RK), R18.2; no longer D10.3 (RK)
- net D+: now also R4.2, U2.5 (D+)
- net D-: now also R3.2, U2.4 (D-)
- net DC/SA0_3.3V: now also JP4.2 (B)
- net ENCODER_A1: now also SW1.A, U2.61 (PF0)
- net ENCODER_A2: now also U2.59 (PF2)
- net ENCODER_B1: now also SW1.B, U2.60 (PF1)
- net ENCODER_B2: now also U2.58 (PF3)
- net GND: now also U3.13 (/CS), C1.2, C10.2, C11.2, C12.2, C13.2, C14.2, C15.1, C17.1, C19.2, C2.1, C20.2, C21.2, C22.2, C23.2, C3.2, C4.2, C5.2, C6.1, C7.2, C8.2, C9.2, D8.1 (K), IC1.12 (GND), IC1.36 (GND), IC1.55 (GND), IC1.8 (ADDR), JP4.1 (A), R19.2, R21.2, R22.2, R23.2, R24.2, R5.1, R6.1, R7.1, SW1.C, SW2.1, U2.22 (GND), U2.53 (GND), U2.6 (UGND), U2.63 (GND), U4.2 (GND), USB-C1.A1 (GND), USB-C1.A12 (GND), USB-C1.B1 (GND), USB-C1.B12 (GND), Y1.2, Y1.4; no longer U3.10 (BS0), U3.12 (BS2)
- net MISO: now also U2.13 (PB3)
- net MOSI: now also U2.12 (PB2)
- net RESET: now also R2.2, SW2.2, U2.20 (~{RESET})
- net SCK: now also U2.11 (PB1)
- net SCL: now also IC1.10 (SCL), Q2.3 (D), R9.2, U2.25 (PD0)
- net SCL_3.3: now also Q2.2 (S), R11.2
- net SDA: now also IC1.9 (SDA), Q1.3 (D), R10.2, U2.26 (PD1)
- net SDA_3.3: now also JP5.1 (A), Q1.2 (S), R12.2
- net SW1: now also D11.4 (A), D9.4 (A), IC1.16 (SW1); no longer D10.4 (A)
- net SW2: now also D10.4 (A), D12.4 (A), IC1.17 (SW2); no longer D11.4 (A)
- net VCC: now also F1.1, J1.2 (VCC), U3.28 (VCC), C23.1, R1.1, USB-C1.A4 (VBUS), USB-C1.A9 (VBUS), USB-C1.B4 (VBUS), USB-C1.B9 (VBUS); no longer F1.2
- net XTAL1: now also C2.2, U2.24 (XTAL1), Y1.1
- net XTAL2: now also C6.2, U2.23 (XTAL2), Y1.3
- net at MX4.2 (ROW): now also D6.2 (A)
- net at D1.2 (A): now also R1.2
- net VCOMH: now reaches U3.27 (VCOMH)
- net VCOMH: now also C22.1
- net at U1.2 (IO1): now also R4.1, USB-C1.A6 (D+), USB-C1.B6 (D+)
- net at U1.3 (IO2): now also R3.1, USB-C1.A7 (D-), USB-C1.B7 (D-)
- net C1N: now reaches U3.5 (C1N)
- net C1N: now also C18.2
- net C1P: now reaches U3.4 (C1P)
- net C1P: now also C18.1
- net at SW3.S2: now also D7.2 (A)
- net at MX3.2 (ROW): now also D5.2 (A)
- net at MX2.2 (ROW): now also D3.2 (A)
- net C2N: now reaches U3.3 (C2N)
- net C2N: now also C16.2
- net C2P: now reaches U3.2 (C2P)
- net C2P: now also C16.1
- net D2/SDA: now reaches U3.20 (D2/I2C_SDA)
- net D2/SDA: now also JP5.2 (B)
- net IREF: now reaches U3.26 (IREF)
- net IREF: now also R24.1
- net at MX1.2 (ROW): now also D2.2 (A)
- net 3.3V renamed +3V3
- net +3V3: now also C15.2, C17.2, C4.1, C5.1, JP1.1 (A), JP2.1 (A), JP3.1 (A), Q1.1 (G), Q2.1 (G), R11.1, R12.1, R8.1, U4.5 (VOUT); no longer U3.11 (BS1)
- new net: D4.2 (A), SW1.S2
- new net: C21.1, IC1.11 (SDB), R20.2
- new net: IC1.27 (CS02), R14.1
- new net: R5.2, USB-C1.B5 (CC2)
- new net: IC1.31 (CS06), R18.1
- new net: D8.2 (A), R8.2
- new net: IC1.13 (ISET), R22.1
- new net: IC1.26 (CS01), R13.1
- new net: IC1.30 (CS05), R17.1
- new net: R7.2, U2.43 (PE2/~{HWB})
- new net: R6.2, USB-C1.A5 (CC1)
- new net: C1.1, U2.7 (UCAP)
- new net: IC1.28 (CS03), R15.1
- new net: IC1.29 (CS04), R16.1
- new net BS0: JP1.2 (B), R19.1, U3.10 (BS0)
- new net BS1: JP2.2 (B), R21.1, U3.11 (BS1)
- new net BS2: JP3.2 (B), R23.1, U3.12 (BS2)
- new net ROW0: D2.1 (K), D3.1 (K), D4.1 (K), U2.34 (PE1)
- new net ROW1: D5.1 (K), D6.1 (K), D7.1 (K), U2.33 (PE0)
- no-connect marks 37 -> 84
Other:
- note removed: "D"
- note removed: "G"
- note removed: "I2C"
- note removed: "Keyboard keys LED"
- note removed: "Open for"
- note removed: "S"

Commit message: Start working on pcb
Parts:
- JP1, JP2, JP3, JP4: footprint ProtoFull_Project Libs:SolderJumper-2_P1.3mm_Open_RoundedPad1.0x1.5mm -> SamacSys_Parts:SolderJumper-2_P1.3mm_Open_RoundedPad1.0x1.5mm
- JP5: footprint ProtoFull_Project Libs:SolderJumper-2_P1.3mm_Bridged_RoundedPad1.0x1.5mm -> SamacSys_Parts:SolderJumper-2_P1.3mm_Bridged_RoundedPad1.0x1.5mm
Connections:
- net +3V3: now also C23.1, U3.28 (VCC)
- net +5V: now also J1.2 (VCC)
- net VCC: no longer C23.1, J1.2 (VCC), U3.28 (VCC)
Changed lines of the file:
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@@
     (effects (font (size 1.2446 1.2446)) (justify left bottom))
   )
-  (label "VCC" (at 79.375 384.175 0)
+  (label "+3V3" (at 79.375 384.175 0)
     (effects (font (size 1.27 1.27)) (justify left bottom))
   )
@@
     (effects (font (size 1.27 1.27)) (justify left bottom))
   )
-  (label "VCC" (at 70.485 384.175 0)
+  (label "+3V3" (at 70.485 384.175 0)
     (effects (font (size 1.27 1.27)) (justify left bottom))
   )
@@
     )
     (property "Value" "I2C" (id 1) (at 61.595 363.855 0))
-    (property "Footprint" "ProtoFull_Project Libs:SolderJumper-2_P1.3mm_Bridged_RoundedPad1.0x1.5mm" (id 2) (at 61.595 366.395 0)
+    (property "Footprint" "SamacSys_Parts:SolderJumper-2_P1.3mm_Bridged_RoundedPad1.0x1.5mm" (id 2) (at 61.595 366.395 0)
       (effects (font (size 1.27 1.27)) hide)
     )
@@
     (pin "2")
   )
+  (symbol (lib_id "power:+5V") (at 139.065 27.305 0) (unit 1)
+    (in_bom yes) (on_board yes) (fields_autoplaced)
+    (property "Reference" "#PWR0105" (id 0) (at 139.065 31.115 0)
+      (effects (font (size 1.27 1.27)) hide)
+    )
+    (property "Value" "+5V" (id 1) (at 141.605 26.0349 0)
+      (effects (font (size 1.27 1.27)) (justify left))
+    )
+    (property "Footprint" "" (id 2) (at 139.065 27.305 0)
+      (effects (font (size 1.27 1.27)) hide)
+    )
+    (property "Datasheet" "" (id 3) (at 139.065 27.305 0)
+      (effects (font (size 1.27 1.27)) hide)
+    )
+    (pin "1")
+  )
   (symbol (lib_id "Device:R") (at 243.205 164.465 90) (unit 1)
     (in_bom yes) (on_board yes)
@@
     )
     (property "Value" "BS2" (id 1) (at 34.925 330.835 0))
-    (property "Footprint" "ProtoFull_Project Libs:SolderJumper-2_P1.3mm_Open_RoundedPad1.0x1.5mm" (id 2) (at 34.925 333.375 0)
+    (property "Footprint" "SamacSys_Parts:SolderJumper-2_P1.3mm_Open_RoundedPad1.0x1.5mm" (id 2) (at 34.925 333.375 0)
       (effects (font (size 1.27 1.27)) hide)
     )
@@
     )
     (property "Value" "BS1" (id 1) (at 34.925 325.755 0))
-    (property "Footprint" "ProtoFull_Project Libs:SolderJumper-2_P1.3mm_Open_RoundedPad1.0x1.5mm" (id 2) (at 34.925 328.295 0)
+    (property "Footprint" "SamacSys_Parts:SolderJumper-2_P1.3mm_Open_RoundedPad1.0x1.5mm" (id 2) (at 34.925 328.295 0)
       (effects (font (size 1.27 1.27)) hide)
     )
@@
     )
     (property "Value" "SA0" (id 1) (at 55.245 351.155 0))
-    (property "Footprint" "ProtoFull_Project Libs:SolderJumper-2_P1.3mm_Open_RoundedPad1.0x1.5mm" (id 2) (at 55.245 353.695 0)
+    (property "Footprint" "SamacSys_Parts:SolderJumper-2_P1.3mm_Open_RoundedPad1.0x1.5mm" (id 2) (at 55.245 353.695 0)
       (effects (font (size 1.27 1.27)) hide)
     )
@@
     (pin "1")
   )
-  (symbol (lib_id "power:VCC") (at 139.065 27.305 0) (unit 1)
-    (in_bom yes) (on_board yes) (fields_autoplaced)
-    (property "Reference" "#PWR05" (id 0) (at 139.065 31.115 0)
-      (effects (font (size 1.27 1.27)) hide)
-    )
-    (property "Value" "VCC" (id 1) (at 139.065 22.225 0))
-    (property "Footprint" "" (id 2) (at 139.065 27.305 0)
-      (effects (font (size 1.27 1.27)) hide)
-    )
-    (property "Datasheet" "" (id 3) (at 139.065 27.305 0)
-      (effects (font (size 1.27 1.27)) hide)
-    )
-    (pin "1")
-  )
   (symbol (lib_id "power:GND") (at 184.785 53.975 0) (unit 1)
     (in_bom yes) (on_board yes)
@@
     )
     (property "Value" "BS0" (id 1) (at 34.925 320.675 0))
-    (property "Footprint" "ProtoFull_Project Libs:SolderJumper-2_P1.3mm_Open_RoundedPad1.0x1.5mm" (id 2) (at 34.925 323.215 0)
+    (property "Footprint" "SamacSys_Parts:SolderJumper-2_P1.3mm_Open_RoundedPad1.0x1.5mm" (id 2) (at 34.925 323.215 0)
       (effects (font (size 1.27 1.27)) hide)
     )
@@
       (reference "#PWR04") (unit 1) (value "+5V") (footprint "")
     )
-    (path "/e36784ed-e766-4211-8d29-68b2c0bc0e72"
-      (reference "#PWR05") (unit 1) (value "VCC") (footprint "")
-    )
     (path "/ef51adb2-ff9e-4002-a0aa-e8b44dda867d"
       (reference "#PWR06") (unit 1) (value "GND") (footprint "")
@@
       (reference "#PWR0104") (unit 1) (value "+3V3") (footprint "")
     )
+    (path "/3b7cbf4a-aa4b-412f-a33f-2d22918830fe"
+      (reference "#PWR0105") (unit 1) (value "+5V") (footprint "")
+    )
     (path "/aab7d87d-7003-4bc7-942c-682e6a360e6f"
       (reference "C1") (unit 1) (value "1uF") (footprint "Capacitor_SMD:C_0805_2012Metric")
@@
     )
     (path "/e7df2dcc-0a1b-497c-8292-c406cecf4343"
-      (reference "JP1") (unit 1) (value "BS0") (footprint "ProtoFull_Project Libs:SolderJumper-2_P1.3mm_Open_RoundedPad1.0x1.5mm")
+      (reference "JP1") (unit 1) (value "BS0") (footprint "SamacSys_Parts:SolderJumper-2_P1.3mm_Open_RoundedPad1.0x1.5mm")
     )
     (path "/b8374e86-f9f1-4ee5-b573-4a17c9ee7ecc"
-      (reference "JP2") (unit 1) (value "BS1") (footprint "ProtoFull_Project Libs:SolderJumper-2_P1.3mm_Open_RoundedPad1.0x1.5mm")
+      (reference "JP2") (unit 1) (value "BS1") (footprint "SamacSys_Parts:SolderJumper-2_P1.3mm_Open_RoundedPad1.0x1.5mm")
     )
     (path "/86476e84-6914-498e-a9f3-3e0b63c65e24"
-      (reference "JP3") (unit 1) (value "BS2") (footprint "ProtoFull_Project Libs:SolderJumper-2_P1.3mm_Open_RoundedPad1.0x1.5mm")
+      (reference "JP3") (unit 1) (value "BS2") (footprint "SamacSys_Parts:SolderJumper-2_P1.3mm_Open_RoundedPad1.0x1.5mm")
     )
     (path "/d7bf7d66-8b84-4a42-bbff-8720f69fe3dd"
-      (reference "JP4") (unit 1) (value "SA0") (footprint "ProtoFull_Project Libs:SolderJumper-2_P1.3mm_Open_RoundedPad1.0x1.5mm")
+      (reference "JP4") (unit 1) (value "SA0") (footprint "SamacSys_Parts:SolderJumper-2_P1.3mm_Open_RoundedPad1.0x1.5mm")
     )
     (path "/245799d1-29c3-40de-809d-b7d8ffe59331"
-      (reference "JP5") (unit 1) (value "I2C") (footprint "ProtoFull_Project Libs:SolderJumper-2_P1.3mm_Bridged_RoundedPad1.0x1.5mm")
+      (reference "JP5") (unit 1) (value "I2C") (footprint "SamacSys_Parts:SolderJumper-2_P1.3mm_Bridged_RoundedPad1.0x1.5mm")
     )
     (path "/adc07a0d-20d0-401e-9139-c0df1171be5e"
